File: pedals/distortion/kicad/Flashover/controls.kicad_sch (KiCad schematic)
At the start: 20 parts, among them SW1 PEC11R-4215F-S0024, SW2 PEC11R-4215F-S0024, SW3 PEC11R-4215F-S0024, SW4 Soft/Hard

Commit message: Assign Flashover footprints
Surface-mount for assembly; through-hole for jacks, encoders, panel LEDs,
the Soft/Hard button, the TO-220 regulator and the germanium diodes.
Q1/Q2 use the MMBT3904 symbol, 1N4148 -> 1N4148W, 1N5817 -> SS14.

Co-Authored-By: Claude Opus 5.5 <noreply@anthropic.com>
Parts:
- C33, C34, C35, C36, C37, C38: footprint (none) -> Capacitor_SMD:C_0805_2012Metric
- R23, R24, R25, R26, R27, R28, R29, R30, R31, R32: footprint (none) -> Resistor_SMD:R_0805_2012Metric
- SW1, SW2, SW3: footprint (none) -> Rotary_Encoder:RotaryEncoder_Alps_EC11E-Switch_Vertical_H20mm
- SW4: footprint (none) -> Button_Switch_THT:SW_PUSH_6mm_H13mm
