File: pedals/distortion/kicad/Flashover/led_rings.kicad_sch (KiCad schematic)
At the start: 43 parts, among them U10 IS31FL3236A

Commit message: Apply datasheet checks to Flashover
R33 = 15k (about 5 mA per LED, from the IS31FL3236A current formula).
R39 marked 33 ohm 0.5W per MIDI CA-033. R4 390 -> 330 because the
MCP45HV51 wiper resistance is about 150 ohms at 9V (below its 10V
specified range); sim model Rw updated to match. Pot symbol description
corrected to 8-bit. Product document records the check results.

Co-Authored-By: Claude Opus 5.5 <noreply@anthropic.com>
Parts:
- R33: value R_EXT -> 15k
Other:
- note added: "R33 sets the maximum LED current: 58.5 x 1.3V / R33 = about 5 mA. Firmware can scale it down and dim with PWM."
- note removed: "R33 sets the maximum LED current (about 5 mA); value from the datasheet"

Commit message: Assign Flashover footprints
Surface-mount for assembly; through-hole for jacks, encoders, panel LEDs,
the Soft/Hard button, the TO-220 regulator and the germanium diodes.
Q1/Q2 use the MMBT3904 symbol, 1N4148 -> 1N4148W, 1N5817 -> SS14.

Co-Authored-By: Claude Opus 5.5 <noreply@anthropic.com>
Parts:
- C39, C40: footprint (none) -> Capacitor_SMD:C_0805_2012Metric
- D10, D11, D12, D13, D14, D15, D16, D17, D18, D19, D20, D21, D22, D23, D24, D25, D26, D27, D28, D29, D30, D31, D32, D33, D34, D35, D36, D37, D38, D39, D7, D8, D9: footprint (none) -> LED_SMD:LED_0805_2012Metric
- D40, D41, D42: footprint (none) -> LED_THT:LED_D3.0mm
- R33, R34, R35, R36: footprint (none) -> Resistor_SMD:R_0805_2012Metric
- U10: footprint (none) -> Package_QFP:TQFP-48-1EP_7x7mm_P0.5mm_EP4.11x4.11mm
