File: pedals/distortion/kicad/Flashover/clipping.kicad_sch (KiCad schematic)
At the start: 13 parts, among them K1 G6K-2F-Y 5VDC, Q1 MMBT3904

Commit message: Assign Flashover footprints
Surface-mount for assembly; through-hole for jacks, encoders, panel LEDs,
the Soft/Hard button, the TO-220 regulator and the germanium diodes.
Q1/Q2 use the MMBT3904 symbol, 1N4148 -> 1N4148W, 1N5817 -> SS14.

Co-Authored-By: Claude Opus 5.5 <noreply@anthropic.com>
Parts:
- removed Q1: MMBT3904, symbol Device:Q_NPN
- added Q1: MMBT3904, Package_TO_SOT_SMD:SOT-23, symbol Transistor_BJT:MMBT3904
- C4: footprint (none) -> Capacitor_SMD:C_1210_3225Metric
- C5: footprint (none) -> Capacitor_SMD:C_0805_2012Metric
- D1, D2: footprint (none) -> Diode_THT:D_DO-35_SOD27_P7.62mm_Horizontal
- D4, D5, D6: value 1N4148 -> 1N4148W; footprint (none) -> Diode_SMD:D_SOD-123
- K1: footprint (none) -> Relay_SMD:Relay_DPDT_Omron_G6K-2F-Y
- R10, R12, R13, R6: footprint (none) -> Resistor_SMD:R_0805_2012Metric
Connections:
- net GND: now also Q1.2 (E)
- net at R12.1, R13.1: now also Q1.1 (B)
- net at D6.2 (A), K1.8: now also Q1.3 (C)
Changed lines of the file:
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@@
 			(effects (font (size 1.27 1.27)))
 		)
-		(property "Footprint" ""
+		(property "Footprint" "Capacitor_SMD:C_1210_3225Metric"
 			(at 35.56 68.58 90)
 			(hide yes)
@@
 		(instances
 			(project "Flashover"
-				(path "/d341370c-bf24-48b8-b9fb-db9600491445/c22cd9a2-81b9-45fd-8fd2-6181600e4d84"
+				(path "/872055d3-e01a-4a82-8c05-28c93674a700/06cc9006-e4d3-46e5-abbb-6442b648b186"
 					(reference "C4")
 					(unit 1)
@@
 			(effects (font (size 1.27 1.27)))
 		)
-		(property "Footprint" ""
+		(property "Footprint" "Resistor_SMD:R_0805_2012Metric"
 			(at 46.99 68.58 90)
 			(hide yes)
@@
 		(instances
 			(project "Flashover"
-				(path "/d341370c-bf24-48b8-b9fb-db9600491445/c22cd9a2-81b9-45fd-8fd2-6181600e4d84"
+				(path "/872055d3-e01a-4a82-8c05-28c93674a700/06cc9006-e4d3-46e5-abbb-6442b648b186"
 					(reference "R6")
 					(unit 1)
@@
 			(effects (font (size 1.27 1.27)) (justify left))
 		)
-		(property "Footprint" ""
+		(property "Footprint" "Relay_SMD:Relay_DPDT_Omron_G6K-2F-Y"
 			(at 111.76 83.82 0)
 			(hide yes)
@@
 		(instances
 			(project "Flashover"
-				(path "/d341370c-bf24-48b8-b9fb-db9600491445/c22cd9a2-81b9-45fd-8fd2-6181600e4d84"
+				(path "/872055d3-e01a-4a82-8c05-28c93674a700/06cc9006-e4d3-46e5-abbb-6442b648b186"
 					(reference "K1")
 					(unit 1)
@@
 			(effects (font (size 1.27 1.27)) (justify left))
 		)
-		(property "Footprint" ""
+		(property "Footprint" "Resistor_SMD:R_0805_2012Metric"
 			(at 60.96 77.47 0)
 			(hide yes)
@@
 		(instances
 			(project "Flashover"
-				(path "/d341370c-bf24-48b8-b9fb-db9600491445/c22cd9a2-81b9-45fd-8fd2-6181600e4d84"
+				(path "/872055d3-e01a-4a82-8c05-28c93674a700/06cc9006-e4d3-46e5-abbb-6442b648b186"
 					(reference "R10")
 					(unit 1)
@@
 		(instances
 			(project "Flashover"
-				(path "/d341370c-bf24-48b8-b9fb-db9600491445/c22cd9a2-81b9-45fd-8fd2-6181600e4d84"
+				(path "/872055d3-e01a-4a82-8c05-28c93674a700/06cc9006-e4d3-46e5-abbb-6442b648b186"
 					(reference "#PWR09")
 					(unit 1)
@@
 			(effects (font (size 1.27 1.27)) (justify left))
 		)
-		(property "Footprint" ""
+		(property "Footprint" "Capacitor_SMD:C_0805_2012Metric"
 			(at 68.58 77.47 0)
 			(hide yes)
@@
 		(instances
 			(project "Flashover"
-				(path "/d341370c-bf24-48b8-b9fb-db9600491445/c22cd9a2-81b9-45fd-8fd2-6181600e4d84"
+				(path "/872055d3-e01a-4a82-8c05-28c93674a700/06cc9006-e4d3-46e5-abbb-6442b648b186"
 					(reference "C5")
 					(unit 1)
@@
 		(instances
 			(project "Flashover"
-				(path "/d341370c-bf24-48b8-b9fb-db9600491445/c22cd9a2-81b9-45fd-8fd2-6181600e4d84"
+				(path "/872055d3-e01a-4a82-8c05-28c93674a700/06cc9006-e4d3-46e5-abbb-6442b648b186"
 					(reference "#PWR10")
 					(unit 1)
@@
 			(effects (font (size 1.27 1.27)))
 		)
-		(property "Footprint" ""
+		(property "Footprint" "Diode_THT:D_DO-35_SOD27_P7.62mm_Horizontal"
 			(at 114.3 102.87 90)
 			(hide yes)
@@
 		(instances
 			(project "Flashover"
-				(path "/d341370c-bf24-48b8-b9fb-db9600491445/c22cd9a2-81b9-45fd-8fd2-6181600e4d84"
+				(path "/872055d3-e01a-4a82-8c05-28c93674a700/06cc9006-e4d3-46e5-abbb-6442b648b186"
 					(reference "D1")
 					(unit 1)
@@
 			(effects (font (size 1.27 1.27)))
 		)
-		(property "Footprint" ""
+		(property "Footprint" "Diode_THT:D_DO-35_SOD27_P7.62mm_Horizontal"
 			(at 104.14 102.87 270)
 			(hide yes)
@@
 		(instances
 			(project "Flashover"
-				(path "/d341370c-bf24-48b8-b9fb-db9600491445/c22cd9a2-81b9-45fd-8fd2-6181600e4d84"
+				(path "/872055d3-e01a-4a82-8c05-28c93674a700/06cc9006-e4d3-46e5-abbb-6442b648b186"
 					(reference "D2")
 					(unit 1)
@@
 		(instances
 			(project "Flashover"
-				(path "/d341370c-bf24-48b8-b9fb-db9600491445/c22cd9a2-81b9-45fd-8fd2-6181600e4d84"
+				(path "/872055d3-e01a-4a82-8c05-28c93674a700/06cc9006-e4d3-46e5-abbb-6442b648b186"
 					(reference "#PWR11")
 					(unit 1)
@@
 			(effects (font (size 1.27 1.27)))
 		)
-		(property "Value" "1N4148"
-			(at 93.091 104.14 90)
-			(show_name no)
-			(do_not_autoplace no)
-			(effects (font (size 1.27 1.27)))
-		)
-		(property "Footprint" ""
+		(property "Value" "1N4148W"
+			(at 92.5195 104.14 90)
+			(show_name no)
+			(do_not_autoplace no)
+			(effects (font (size 1.27 1.27)))
+		)
+		(property "Footprint" "Diode_SMD:D_SOD-123"
 			(at 99.06 102.87 90)
 			(hide yes)
@@
 		(instances
 			(project "Flashover"
-				(path "/d341370c-bf24-48b8-b9fb-db9600491445/c22cd9a2-81b9-45fd-8fd2-6181600e4d84"
+				(path "/872055d3-e01a-4a82-8c05-28c93674a700/06cc9006-e4d3-46e5-abbb-6442b648b186"
 					(reference "D4")
 					(unit 1)
@@
 			(effects (font (size 1.27 1.27)))
 		)
-		(property "Value" "1N4148"
-			(at 80.391 104.14 270)
-			(show_name no)
-			(do_not_autoplace no)
-			(effects (font (size 1.27 1.27)))
-		)
-		(property "Footprint" ""
+		(property "Value" "1N4148W"
+			(at 79.8195 104.14 270)
+			(show_name no)
+			(do_not_autoplace no)
+			(effects (font (size 1.27 1.27)))
+		)
+		(property "Footprint" "Diode_SMD:D_SOD-123"
 			(at 86.36 102.87 270)
 			(hide yes)
@@
 		(instances
 			(project "Flashover"
-				(path "/d341370c-bf24-48b8-b9fb-db9600491445/c22cd9a2-81b9-45fd-8fd2-6181600e4d84"
+				(path "/872055d3-e01a-4a82-8c05-28c93674a700/06cc9006-e4d3-46e5-abbb-6442b648b186"
 					(reference "D5")
 					(unit 1)
@@
 		(instances
 			(project "Flashover"
-				(path "/d341370c-bf24-48b8-b9fb-db9600491445/c22cd9a2-81b9-45fd-8fd2-6181600e4d84"
+				(path "/872055d3-e01a-4a82-8c05-28c93674a700/06cc9006-e4d3-46e5-abbb-6442b648b186"
 					(reference "#PWR12")
 					(unit 1)
@@
 			(effects (font (size 1.27 1.27)))
 		)
-		(property "Value" "1N4148"
-			(at 132.969 85.09 90)
-			(show_name no)
-			(do_not_autoplace no)
-			(effects (font (size 1.27 1.27)))
-		)
-		(property "Footprint" ""
+		(property "Value" "1N4148W"
+			(at 133.5405 85.09 90)
+			(show_name no)
+			(do_not_autoplace no)
+			(effects (font (size 1.27 1.27)))
+		)
+		(property "Footprint" "Diode_SMD:D_SOD-123"
 			(at 127 83.82 90)
 			(hide yes)
@@
 		(instances
 			(project "Flashover"
-				(path "/d341370c-bf24-48b8-b9fb-db9600491445/c22cd9a2-81b9-45fd-8fd2-6181600e4d84"
+				(path "/872055d3-e01a-4a82-8c05-28c93674a700/06cc9006-e4d3-46e5-abbb-6442b648b186"
 					(reference "D6")
 					(unit 1)
@@
 	)
 	(symbol
-		(lib_id "Device:Q_NPN")
+		(lib_id "Transistor_BJT:MMBT3904")
 		(at 147.32 101.6 0)
 		(mirror y)
@@
 			(effects (font (size 1.27 1.27)))
 		)
-		(property "Footprint" ""
+		(property "Footprint" "Package_TO_SOT_SMD:SOT-23"
 			(at 147.32 101.6 0)
 			(hide yes)
@@
 			(effects (font (size 1.27 1.27)))
 		)
-		(pin "B"
-		)
-		(pin "C"
-		)
-		(pin "E"
-		)
-		(instances
-			(project "Flashover"
-				(path "/d341370c-bf24-48b8-b9fb-db9600491445/c22cd9a2-81b9-45fd-8fd2-6181600e4d84"
+		(pin "1"
+		)
+		(pin "2"
+		)
+		(pin "3"
+		)
+		(instances
+			(project "Flashover"
+				(path "/872055d3-e01a-4a82-8c05-28c93674a700/06cc9006-e4d3-46e5-abbb-6442b648b186"
 					(reference "Q1")
 					(unit 1)
@@
 		(instances
 			(project "Flashover"
-				(path "/d341370c-bf24-48b8-b9fb-db9600491445/c22cd9a2-81b9-45fd-8fd2-6181600e4d84"
+				(path "/872055d3-e01a-4a82-8c05-28c93674a700/06cc9006-e4d3-46e5-abbb-6442b648b186"
 					(reference "#PWR13")
 					(unit 1)
@@
 		(instances
 			(project "Flashover"
-				(path "/d341370c-bf24-48b8-b9fb-db9600491445/c22cd9a2-81b9-45fd-8fd2-6181600e4d84"
+				(path "/872055d3-e01a-4a82-8c05-28c93674a700/06cc9006-e4d3-46e5-abbb-6442b648b186"
 					(reference "#PWR14")
 					(unit 1)
@@
 			(effects (font (size 1.27 1.27)))
 		)
-		(property "Footprint" ""
+		(property "Footprint" "Resistor_SMD:R_0805_2012Metric"
 			(at 160.02 101.6 90)
 			(hide yes)
@@
 		(instances
 			(project "Flashover"
-				(path "/d341370c-bf24-48b8-b9fb-db9600491445/c22cd9a2-81b9-45fd-8fd2-6181600e4d84"
+				(path "/872055d3-e01a-4a82-8c05-28c93674a700/06cc9006-e4d3-46e5-abbb-6442b648b186"
 					(reference "R12")
 					(unit 1)
@@
 			(effects (font (size 1.27 1.27)) (justify left))
 		)
-		(property "Footprint" ""
+		(property "Footprint" "Resistor_SMD:R_0805_2012Metric"
 			(at 153.67 107.95 0)
 			(hide yes)
@@
 		(instances
 			(project "Flashover"
-				(path "/d341370c-bf24-48b8-b9fb-db9600491445/c22cd9a2-81b9-45fd-8fd2-6181600e4d84"
+				(path "/872055d3-e01a-4a82-8c05-28c93674a700/06cc9006-e4d3-46e5-abbb-6442b648b186"
 					(reference "R13")
 					(unit 1)
@@
 		(instances
 			(project "Flashover"
-				(path "/d341370c-bf24-48b8-b9fb-db9600491445/c22cd9a2-81b9-45fd-8fd2-6181600e4d84"
+				(path "/872055d3-e01a-4a82-8c05-28c93674a700/06cc9006-e4d3-46e5-abbb-6442b648b186"
 					(reference "#PWR15")
 					(unit 1)
