File: pedals/distortion/kicad/Flashover/input_gain.kicad_sch (KiCad schematic)
At the start: 12 parts, among them J1 Input, U1 LM741

Commit message: Add Flashover controller and digital pot sheets
Controller sheet: RP2040 with 3.3V regulator, 2 MB QSPI flash, 12 MHz
crystal and SWD header, plus a GPIO plan for the sheets still to come.
Digital Pots sheet: control side of three MCP45HV51 I2C pots with
pull-ups. RV1-RV3 on the audio sheets become the pot units of U7-U9
(new two-unit MCP45HV51 symbol in the shared library). ERC clean.

Co-Authored-By: Claude Opus 5.5 <noreply@anthropic.com>
Parts:
- removed RV1: 100k digital, symbol Device:R_Potentiometer
- added U7: MCP45HV51-104, symbol GreywireStudio:MCP45HV51
Connections:
- net at R4.2: now also U7.13
- net at C3.1: now also U7.11, U7.12
Other:
- note added: "Gain = 1 + R5 / (R4 + U7A): about 2x (min) to 216x (max) U7A is the Gain knob: the pot side of an MCP45HV51 digital pot (100k). Its control and power pins (U7B) are on the Digital Pots sheet."
- note removed: "Gain = 1 + R5 / (R4 + RV1): about 2x (min) to 216x (max) RV1 is one channel of an MCP41HV digital pot (Gain knob). Its control side (SPI) goes on the controller sheet."
Changed lines of the file:
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@@
 		(effects (font (size 1.27 1.27)) (justify left))
 	)
-	(text "Gain = 1 + R5 / (R4 + RV1):  about 2x (min) to 216x (max)\nRV1 is one channel of an MCP41HV digital pot (Gain knob).\nIts control side (SPI) goes on the controller sheet."
+	(text "Gain = 1 + R5 / (R4 + U7A):  about 2x (min) to 216x (max)\nU7A is the Gain knob: the pot side of an MCP45HV51 digital pot (100k).\nIts control and power pins (U7B) are on the Digital Pots sheet."
 		(exclude_from_sim no)
 		(at 20.32 157.48 0)
@@
 		(instances
 			(project "Flashover"
-				(path "/c1c20152-b132-4e14-97dc-1ac24480e45d/d8b4aca9-ddeb-4c76-a690-0335c0a19397"
+				(path "/37bda491-c0dc-4d48-acdf-49df4f139bb0/2e16fd56-5524-4d37-91fb-235b8f173ecd"
 					(reference "J1")
 					(unit 1)
@@
 		(instances
 			(project "Flashover"
-				(path "/c1c20152-b132-4e14-97dc-1ac24480e45d/d8b4aca9-ddeb-4c76-a690-0335c0a19397"
+				(path "/37bda491-c0dc-4d48-acdf-49df4f139bb0/2e16fd56-5524-4d37-91fb-235b8f173ecd"
 					(reference "#PWR01")
 					(unit 1)
@@
 		(instances
 			(project "Flashover"
-				(path "/c1c20152-b132-4e14-97dc-1ac24480e45d/d8b4aca9-ddeb-4c76-a690-0335c0a19397"
+				(path "/37bda491-c0dc-4d48-acdf-49df4f139bb0/2e16fd56-5524-4d37-91fb-235b8f173ecd"
 					(reference "R1")
 					(unit 1)
@@
 		(instances
 			(project "Flashover"
-				(path "/c1c20152-b132-4e14-97dc-1ac24480e45d/d8b4aca9-ddeb-4c76-a690-0335c0a19397"
+				(path "/37bda491-c0dc-4d48-acdf-49df4f139bb0/2e16fd56-5524-4d37-91fb-235b8f173ecd"
 					(reference "#PWR02")
 					(unit 1)
@@
 		(instances
 			(project "Flashover"
-				(path "/c1c20152-b132-4e14-97dc-1ac24480e45d/d8b4aca9-ddeb-4c76-a690-0335c0a19397"
+				(path "/37bda491-c0dc-4d48-acdf-49df4f139bb0/2e16fd56-5524-4d37-91fb-235b8f173ecd"
 					(reference "C1")
 					(unit 1)
@@
 		(instances
 			(project "Flashover"
-				(path "/c1c20152-b132-4e14-97dc-1ac24480e45d/d8b4aca9-ddeb-4c76-a690-0335c0a19397"
+				(path "/37bda491-c0dc-4d48-acdf-49df4f139bb0/2e16fd56-5524-4d37-91fb-235b8f173ecd"
 					(reference "R2")
 					(unit 1)
@@
 		(instances
 			(project "Flashover"
-				(path "/c1c20152-b132-4e14-97dc-1ac24480e45d/d8b4aca9-ddeb-4c76-a690-0335c0a19397"
+				(path "/37bda491-c0dc-4d48-acdf-49df4f139bb0/2e16fd56-5524-4d37-91fb-235b8f173ecd"
 					(reference "U1")
 					(unit 1)
@@
 		(instances
 			(project "Flashover"
-				(path "/c1c20152-b132-4e14-97dc-1ac24480e45d/d8b4aca9-ddeb-4c76-a690-0335c0a19397"
+				(path "/37bda491-c0dc-4d48-acdf-49df4f139bb0/2e16fd56-5524-4d37-91fb-235b8f173ecd"
 					(reference "R3")
 					(unit 1)
@@
 		(instances
 			(project "Flashover"
-				(path "/c1c20152-b132-4e14-97dc-1ac24480e45d/d8b4aca9-ddeb-4c76-a690-0335c0a19397"
+				(path "/37bda491-c0dc-4d48-acdf-49df4f139bb0/2e16fd56-5524-4d37-91fb-235b8f173ecd"
 					(reference "#PWR03")
 					(unit 1)
@@
 		(instances
 			(project "Flashover"
-				(path "/c1c20152-b132-4e14-97dc-1ac24480e45d/d8b4aca9-ddeb-4c76-a690-0335c0a19397"
+				(path "/37bda491-c0dc-4d48-acdf-49df4f139bb0/2e16fd56-5524-4d37-91fb-235b8f173ecd"
 					(reference "C2")
 					(unit 1)
@@
 		(instances
 			(project "Flashover"
-				(path "/c1c20152-b132-4e14-97dc-1ac24480e45d/d8b4aca9-ddeb-4c76-a690-0335c0a19397"
+				(path "/37bda491-c0dc-4d48-acdf-49df4f139bb0/2e16fd56-5524-4d37-91fb-235b8f173ecd"
 					(reference "#PWR04")
 					(unit 1)
@@
 		(instances
 			(project "Flashover"
-				(path "/c1c20152-b132-4e14-97dc-1ac24480e45d/d8b4aca9-ddeb-4c76-a690-0335c0a19397"
+				(path "/37bda491-c0dc-4d48-acdf-49df4f139bb0/2e16fd56-5524-4d37-91fb-235b8f173ecd"
 					(reference "#PWR05")
 					(unit 1)
@@
 		(instances
 			(project "Flashover"
-				(path "/c1c20152-b132-4e14-97dc-1ac24480e45d/d8b4aca9-ddeb-4c76-a690-0335c0a19397"
+				(path "/37bda491-c0dc-4d48-acdf-49df4f139bb0/2e16fd56-5524-4d37-91fb-235b8f173ecd"
 					(reference "#PWR06")
 					(unit 1)
@@
 		(instances
 			(project "Flashover"
-				(path "/c1c20152-b132-4e14-97dc-1ac24480e45d/d8b4aca9-ddeb-4c76-a690-0335c0a19397"
+				(path "/37bda491-c0dc-4d48-acdf-49df4f139bb0/2e16fd56-5524-4d37-91fb-235b8f173ecd"
 					(reference "R5")
 					(unit 1)
@@
 		(instances
 			(project "Flashover"
-				(path "/c1c20152-b132-4e14-97dc-1ac24480e45d/d8b4aca9-ddeb-4c76-a690-0335c0a19397"
+				(path "/37bda491-c0dc-4d48-acdf-49df4f139bb0/2e16fd56-5524-4d37-91fb-235b8f173ecd"
 					(reference "R4")
 					(unit 1)
@@
 	)
 	(symbol
-		(lib_id "Device:R_Potentiometer")
+		(lib_id "GreywireStudio:MCP45HV51")
 		(at 90.17 128.27 0)
 		(unit 1)
@@
 		(in_pos_files yes)
 		(dnp no)
-		(property "Reference" "RV1"
-			(at 87.63 127 0)
-			(show_name no)
-			(do_not_autoplace no)
-			(effects (font (size 1.27 1.27)) (justify right))
-		)
-		(property "Value" "100k digital"
-			(at 87.63 129.54 0)
-			(show_name no)
-			(do_not_autoplace no)
-			(effects (font (size 1.27 1.27)) (justify right))
+		(property "Reference" "U7"
+			(at 96.52 127 0)
+			(show_name no)
+			(do_not_autoplace no)
+			(effects (font (size 1.27 1.27)) (justify left))
+		)
+		(property "Value" "MCP45HV51-104"
+			(at 96.52 129.54 0)
+			(show_name no)
+			(do_not_autoplace no)
+			(effects (font (size 1.27 1.27)) (justify left))
 		)
 		(property "Footprint" ""
@@
 			(effects (font (size 1.27 1.27)))
 		)
-		(pin "1"
-		)
-		(pin "2"
-		)
-		(pin "3"
-		)
-		(instances
-			(project "Flashover"
-				(path "/c1c20152-b132-4e14-97dc-1ac24480e45d/d8b4aca9-ddeb-4c76-a690-0335c0a19397"
-					(reference "RV1")
+		(pin "13"
+		)
+		(pin "12"
+		)
+		(pin "11"
+		)
+		(instances
+			(project "Flashover"
+				(path "/37bda491-c0dc-4d48-acdf-49df4f139bb0/2e16fd56-5524-4d37-91fb-235b8f173ecd"
+					(reference "U7")
 					(unit 1)
 				)
@@
 		(instances
 			(project "Flashover"
-				(path "/c1c20152-b132-4e14-97dc-1ac24480e45d/d8b4aca9-ddeb-4c76-a690-0335c0a19397"
+				(path "/37bda491-c0dc-4d48-acdf-49df4f139bb0/2e16fd56-5524-4d37-91fb-235b8f173ecd"
 					(reference "C3")
 					(unit 1)
@@
 		(instances
 			(project "Flashover"
-				(path "/c1c20152-b132-4e14-97dc-1ac24480e45d/d8b4aca9-ddeb-4c76-a690-0335c0a19397"
+				(path "/37bda491-c0dc-4d48-acdf-49df4f139bb0/2e16fd56-5524-4d37-91fb-235b8f173ecd"
 					(reference "#PWR07")
 					(unit 1)
@@
 		(instances
 			(project "Flashover"
-				(path "/c1c20152-b132-4e14-97dc-1ac24480e45d/d8b4aca9-ddeb-4c76-a690-0335c0a19397"
+				(path "/37bda491-c0dc-4d48-acdf-49df4f139bb0/2e16fd56-5524-4d37-91fb-235b8f173ecd"
 					(reference "C10")
 					(unit 1)
@@
 		(instances
 			(project "Flashover"
-				(path "/c1c20152-b132-4e14-97dc-1ac24480e45d/d8b4aca9-ddeb-4c76-a690-0335c0a19397"
+				(path "/37bda491-c0dc-4d48-acdf-49df4f139bb0/2e16fd56-5524-4d37-91fb-235b8f173ecd"
 					(reference "#PWR08")
 					(unit 1)
@@
 		(instances
 			(project "Flashover"
-				(path "/c1c20152-b132-4e14-97dc-1ac24480e45d/d8b4aca9-ddeb-4c76-a690-0335c0a19397"
+				(path "/37bda491-c0dc-4d48-acdf-49df4f139bb0/2e16fd56-5524-4d37-91fb-235b8f173ecd"
 					(reference "#PWR09")
 					(unit 1)

Commit message: Add Flashover bypass sheet; complete schematic
Bypass sheet: fail-safe G6K-2 relay bypass (NC contacts join the jacks
when unpowered), input/output jacks moved here from the audio sheets
(now FX_IN/FX_OUT), relay driver on FX_ON, soft-touch footswitch and
Link LED. Relay coils on K1 and K2 now take +5V on pin 1 (marked +).
Root sheet laid out in four columns. ERC clean.

Co-Authored-By: Claude Opus 5.5 <noreply@anthropic.com>
Parts:
- removed J1: Input, symbol Connector_Audio:AudioJack2
Connections:
- net FX_IN: now reaches C1.1, R1.1
Other:
- note added: "FX_IN comes from the input jack through the bypass relay (Bypass sheet)."

Commit message: Apply datasheet checks to Flashover
R33 = 15k (about 5 mA per LED, from the IS31FL3236A current formula).
R39 marked 33 ohm 0.5W per MIDI CA-033. R4 390 -> 330 because the
MCP45HV51 wiper resistance is about 150 ohms at 9V (below its 10V
specified range); sim model Rw updated to match. Pot symbol description
corrected to 8-bit. Product document records the check results.

Co-Authored-By: Claude Opus 5.5 <noreply@anthropic.com>
Parts:
- R4: value 390 -> 330
Changed lines of the file:
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@@
 		(instances
 			(project "Flashover"
-				(path "/d44d1406-41c8-4e08-862e-64ff4a05b8dc/c3900c17-15a2-424d-8cbd-c2d255d63a5e"
+				(path "/d341370c-bf24-48b8-b9fb-db9600491445/d807c62d-c7b4-41f0-8d75-0f3cff6869c0"
 					(reference "R1")
 					(unit 1)
@@
 		(instances
 			(project "Flashover"
-				(path "/d44d1406-41c8-4e08-862e-64ff4a05b8dc/c3900c17-15a2-424d-8cbd-c2d255d63a5e"
+				(path "/d341370c-bf24-48b8-b9fb-db9600491445/d807c62d-c7b4-41f0-8d75-0f3cff6869c0"
 					(reference "#PWR01")
 					(unit 1)
@@
 		(instances
 			(project "Flashover"
-				(path "/d44d1406-41c8-4e08-862e-64ff4a05b8dc/c3900c17-15a2-424d-8cbd-c2d255d63a5e"
+				(path "/d341370c-bf24-48b8-b9fb-db9600491445/d807c62d-c7b4-41f0-8d75-0f3cff6869c0"
 					(reference "C1")
 					(unit 1)
@@
 		(instances
 			(project "Flashover"
-				(path "/d44d1406-41c8-4e08-862e-64ff4a05b8dc/c3900c17-15a2-424d-8cbd-c2d255d63a5e"
+				(path "/d341370c-bf24-48b8-b9fb-db9600491445/d807c62d-c7b4-41f0-8d75-0f3cff6869c0"
 					(reference "R2")
 					(unit 1)
@@
 		(instances
 			(project "Flashover"
-				(path "/d44d1406-41c8-4e08-862e-64ff4a05b8dc/c3900c17-15a2-424d-8cbd-c2d255d63a5e"
+				(path "/d341370c-bf24-48b8-b9fb-db9600491445/d807c62d-c7b4-41f0-8d75-0f3cff6869c0"
 					(reference "U1")
 					(unit 1)
@@
 		(instances
 			(project "Flashover"
-				(path "/d44d1406-41c8-4e08-862e-64ff4a05b8dc/c3900c17-15a2-424d-8cbd-c2d255d63a5e"
+				(path "/d341370c-bf24-48b8-b9fb-db9600491445/d807c62d-c7b4-41f0-8d75-0f3cff6869c0"
 					(reference "R3")
 					(unit 1)
@@
 		(instances
 			(project "Flashover"
-				(path "/d44d1406-41c8-4e08-862e-64ff4a05b8dc/c3900c17-15a2-424d-8cbd-c2d255d63a5e"
+				(path "/d341370c-bf24-48b8-b9fb-db9600491445/d807c62d-c7b4-41f0-8d75-0f3cff6869c0"
 					(reference "#PWR02")
 					(unit 1)
@@
 		(instances
 			(project "Flashover"
-				(path "/d44d1406-41c8-4e08-862e-64ff4a05b8dc/c3900c17-15a2-424d-8cbd-c2d255d63a5e"
+				(path "/d341370c-bf24-48b8-b9fb-db9600491445/d807c62d-c7b4-41f0-8d75-0f3cff6869c0"
 					(reference "C2")
 					(unit 1)
@@
 		(instances
 			(project "Flashover"
-				(path "/d44d1406-41c8-4e08-862e-64ff4a05b8dc/c3900c17-15a2-424d-8cbd-c2d255d63a5e"
+				(path "/d341370c-bf24-48b8-b9fb-db9600491445/d807c62d-c7b4-41f0-8d75-0f3cff6869c0"
 					(reference "#PWR03")
 					(unit 1)
@@
 		(instances
 			(project "Flashover"
-				(path "/d44d1406-41c8-4e08-862e-64ff4a05b8dc/c3900c17-15a2-424d-8cbd-c2d255d63a5e"
+				(path "/d341370c-bf24-48b8-b9fb-db9600491445/d807c62d-c7b4-41f0-8d75-0f3cff6869c0"
 					(reference "#PWR04")
 					(unit 1)
@@
 		(instances
 			(project "Flashover"
-				(path "/d44d1406-41c8-4e08-862e-64ff4a05b8dc/c3900c17-15a2-424d-8cbd-c2d255d63a5e"
+				(path "/d341370c-bf24-48b8-b9fb-db9600491445/d807c62d-c7b4-41f0-8d75-0f3cff6869c0"
 					(reference "#PWR05")
 					(unit 1)
@@
 		(instances
 			(project "Flashover"
-				(path "/d44d1406-41c8-4e08-862e-64ff4a05b8dc/c3900c17-15a2-424d-8cbd-c2d255d63a5e"
+				(path "/d341370c-bf24-48b8-b9fb-db9600491445/d807c62d-c7b4-41f0-8d75-0f3cff6869c0"
 					(reference "R5")
 					(unit 1)
@@
 			(effects (font (size 1.27 1.27)) (justify left))
 		)
-		(property "Value" "390"
+		(property "Value" "330"
 			(at 92.71 118.11 0)
 			(show_name no)
@@
 		(instances
 			(project "Flashover"
-				(path "/d44d1406-41c8-4e08-862e-64ff4a05b8dc/c3900c17-15a2-424d-8cbd-c2d255d63a5e"
+				(path "/d341370c-bf24-48b8-b9fb-db9600491445/d807c62d-c7b4-41f0-8d75-0f3cff6869c0"
 					(reference "R4")
 					(unit 1)
@@
 		(instances
 			(project "Flashover"
-				(path "/d44d1406-41c8-4e08-862e-64ff4a05b8dc/c3900c17-15a2-424d-8cbd-c2d255d63a5e"
+				(path "/d341370c-bf24-48b8-b9fb-db9600491445/d807c62d-c7b4-41f0-8d75-0f3cff6869c0"
 					(reference "U7")
 					(unit 1)
@@
 		(instances
 			(project "Flashover"
-				(path "/d44d1406-41c8-4e08-862e-64ff4a05b8dc/c3900c17-15a2-424d-8cbd-c2d255d63a5e"
+				(path "/d341370c-bf24-48b8-b9fb-db9600491445/d807c62d-c7b4-41f0-8d75-0f3cff6869c0"
 					(reference "C3")
 					(unit 1)
@@
 		(instances
 			(project "Flashover"
-				(path "/d44d1406-41c8-4e08-862e-64ff4a05b8dc/c3900c17-15a2-424d-8cbd-c2d255d63a5e"
+				(path "/d341370c-bf24-48b8-b9fb-db9600491445/d807c62d-c7b4-41f0-8d75-0f3cff6869c0"
 					(reference "#PWR06")
 					(unit 1)
@@
 		(instances
 			(project "Flashover"
-				(path "/d44d1406-41c8-4e08-862e-64ff4a05b8dc/c3900c17-15a2-424d-8cbd-c2d255d63a5e"
+				(path "/d341370c-bf24-48b8-b9fb-db9600491445/d807c62d-c7b4-41f0-8d75-0f3cff6869c0"
 					(reference "C10")
 					(unit 1)
@@
 		(instances
 			(project "Flashover"
-				(path "/d44d1406-41c8-4e08-862e-64ff4a05b8dc/c3900c17-15a2-424d-8cbd-c2d255d63a5e"
+				(path "/d341370c-bf24-48b8-b9fb-db9600491445/d807c62d-c7b4-41f0-8d75-0f3cff6869c0"
 					(reference "#PWR07")
 					(unit 1)
@@
 		(instances
 			(project "Flashover"
-				(path "/d44d1406-41c8-4e08-862e-64ff4a05b8dc/c3900c17-15a2-424d-8cbd-c2d255d63a5e"
+				(path "/d341370c-bf24-48b8-b9fb-db9600491445/d807c62d-c7b4-41f0-8d75-0f3cff6869c0"
 					(reference "#PWR08")
 					(unit 1)

Commit message: Assign Flashover footprints
Surface-mount for assembly; through-hole for jacks, encoders, panel LEDs,
the Soft/Hard button, the TO-220 regulator and the germanium diodes.
Q1/Q2 use the MMBT3904 symbol, 1N4148 -> 1N4148W, 1N5817 -> SS14.

Co-Authored-By: Claude Opus 5.5 <noreply@anthropic.com>
Parts:
- C1: footprint (none) -> Capacitor_SMD:C_1206_3216Metric
- C10, C2: footprint (none) -> Capacitor_SMD:C_0805_2012Metric
- C3: footprint (none) -> Capacitor_SMD:C_1210_3225Metric
- R1, R2, R3, R4, R5: footprint (none) -> Resistor_SMD:R_0805_2012Metric
- U1: footprint (none) -> Package_SO:SOIC-8_3.9x4.9mm_P1.27mm
- U7: footprint (none) -> Package_SO:TSSOP-14_4.4x5mm_P0.65mm
Changed lines of the file:
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@@
 			(effects (font (size 1.27 1.27)) (justify left))
 		)
-		(property "Footprint" ""
+		(property "Footprint" "Resistor_SMD:R_0805_2012Metric"
 			(at 50.8 96.52 0)
 			(hide yes)
@@
 		(instances
 			(project "Flashover"
-				(path "/d341370c-bf24-48b8-b9fb-db9600491445/d807c62d-c7b4-41f0-8d75-0f3cff6869c0"
+				(path "/872055d3-e01a-4a82-8c05-28c93674a700/1854cea8-bf87-4849-94dd-b39855f3ac8d"
 					(reference "R1")
 					(unit 1)
@@
 		(instances
 			(project "Flashover"
-				(path "/d341370c-bf24-48b8-b9fb-db9600491445/d807c62d-c7b4-41f0-8d75-0f3cff6869c0"
+				(path "/872055d3-e01a-4a82-8c05-28c93674a700/1854cea8-bf87-4849-94dd-b39855f3ac8d"
 					(reference "#PWR01")
 					(unit 1)
@@
 			(effects (font (size 1.27 1.27)))
 		)
-		(property "Footprint" ""
+		(property "Footprint" "Capacitor_SMD:C_1206_3216Metric"
 			(at 58.42 87.63 90)
 			(hide yes)
@@
 		(instances
 			(project "Flashover"
-				(path "/d341370c-bf24-48b8-b9fb-db9600491445/d807c62d-c7b4-41f0-8d75-0f3cff6869c0"
+				(path "/872055d3-e01a-4a82-8c05-28c93674a700/1854cea8-bf87-4849-94dd-b39855f3ac8d"
 					(reference "C1")
 					(unit 1)
@@
 			(effects (font (size 1.27 1.27)))
 		)
-		(property "Footprint" ""
+		(property "Footprint" "Resistor_SMD:R_0805_2012Metric"
 			(at 69.85 87.63 90)
 			(hide yes)
@@
 		(instances
 			(project "Flashover"
-				(path "/d341370c-bf24-48b8-b9fb-db9600491445/d807c62d-c7b4-41f0-8d75-0f3cff6869c0"
+				(path "/872055d3-e01a-4a82-8c05-28c93674a700/1854cea8-bf87-4849-94dd-b39855f3ac8d"
 					(reference "R2")
 					(unit 1)
@@
 			(effects (font (size 1.27 1.27)) (justify left))
 		)
-		(property "Footprint" ""
+		(property "Footprint" "Package_SO:SOIC-8_3.9x4.9mm_P1.27mm"
 			(at 101.6 90.17 0)
 			(hide yes)
@@
 		(instances
 			(project "Flashover"
-				(path "/d341370c-bf24-48b8-b9fb-db9600491445/d807c62d-c7b4-41f0-8d75-0f3cff6869c0"
+				(path "/872055d3-e01a-4a82-8c05-28c93674a700/1854cea8-bf87-4849-94dd-b39855f3ac8d"
 					(reference "U1")
 					(unit 1)
@@
 			(effects (font (size 1.27 1.27)) (justify left))
 		)
-		(property "Footprint" ""
+		(property "Footprint" "Resistor_SMD:R_0805_2012Metric"
 			(at 80.01 78.74 0)
 			(hide yes)
@@
 		(instances
 			(project "Flashover"
-				(path "/d341370c-bf24-48b8-b9fb-db9600491445/d807c62d-c7b4-41f0-8d75-0f3cff6869c0"
+				(path "/872055d3-e01a-4a82-8c05-28c93674a700/1854cea8-bf87-4849-94dd-b39855f3ac8d"
 					(reference "R3")
 					(unit 1)
@@
 		(instances
 			(project "Flashover"
-				(path "/d341370c-bf24-48b8-b9fb-db9600491445/d807c62d-c7b4-41f0-8d75-0f3cff6869c0"
+				(path "/872055d3-e01a-4a82-8c05-28c93674a700/1854cea8-bf87-4849-94dd-b39855f3ac8d"
 					(reference "#PWR02")
 					(unit 1)
@@
 			(effects (font (size 1.27 1.27)) (justify left))
 		)
-		(property "Footprint" ""
+		(property "Footprint" "Capacitor_SMD:C_0805_2012Metric"
 			(at 80.01 96.52 0)
 			(hide yes)
@@
 		(instances
 			(project "Flashover"
-				(path "/d341370c-bf24-48b8-b9fb-db9600491445/d807c62d-c7b4-41f0-8d75-0f3cff6869c0"
+				(path "/872055d3-e01a-4a82-8c05-28c93674a700/1854cea8-bf87-4849-94dd-b39855f3ac8d"
 					(reference "C2")
 					(unit 1)
@@
 		(instances
 			(project "Flashover"
-				(path "/d341370c-bf24-48b8-b9fb-db9600491445/d807c62d-c7b4-41f0-8d75-0f3cff6869c0"
+				(path "/872055d3-e01a-4a82-8c05-28c93674a700/1854cea8-bf87-4849-94dd-b39855f3ac8d"
 					(reference "#PWR03")
 					(unit 1)
@@
 		(instances
 			(project "Flashover"
-				(path "/d341370c-bf24-48b8-b9fb-db9600491445/d807c62d-c7b4-41f0-8d75-0f3cff6869c0"
+				(path "/872055d3-e01a-4a82-8c05-28c93674a700/1854cea8-bf87-4849-94dd-b39855f3ac8d"
 					(reference "#PWR04")
 					(unit 1)
@@
 		(instances
 			(project "Flashover"
-				(path "/d341370c-bf24-48b8-b9fb-db9600491445/d807c62d-c7b4-41f0-8d75-0f3cff6869c0"
+				(path "/872055d3-e01a-4a82-8c05-28c93674a700/1854cea8-bf87-4849-94dd-b39855f3ac8d"
 					(reference "#PWR05")
 					(unit 1)
@@
 			(effects (font (size 1.27 1.27)))
 		)
-		(property "Footprint" ""
+		(property "Footprint" "Resistor_SMD:R_0805_2012Metric"
 			(at 101.6 109.22 90)
 			(hide yes)
@@
 		(instances
 			(project "Flashover"
-				(path "/d341370c-bf24-48b8-b9fb-db9600491445/d807c62d-c7b4-41f0-8d75-0f3cff6869c0"
+				(path "/872055d3-e01a-4a82-8c05-28c93674a700/1854cea8-bf87-4849-94dd-b39855f3ac8d"
 					(reference "R5")
 					(unit 1)
@@
 			(effects (font (size 1.27 1.27)) (justify left))
 		)
-		(property "Footprint" ""
+		(property "Footprint" "Resistor_SMD:R_0805_2012Metric"
 			(at 90.17 116.84 0)
 			(hide yes)
@@
 		(instances
 			(project "Flashover"
-				(path "/d341370c-bf24-48b8-b9fb-db9600491445/d807c62d-c7b4-41f0-8d75-0f3cff6869c0"
+				(path "/872055d3-e01a-4a82-8c05-28c93674a700/1854cea8-bf87-4849-94dd-b39855f3ac8d"
 					(reference "R4")
 					(unit 1)
@@
 			(effects (font (size 1.27 1.27)) (justify left))
 		)
-		(property "Footprint" ""
+		(property "Footprint" "Package_SO:TSSOP-14_4.4x5mm_P0.65mm"
 			(at 90.17 128.27 0)
 			(hide yes)
@@
 		(instances
 			(project "Flashover"
-				(path "/d341370c-bf24-48b8-b9fb-db9600491445/d807c62d-c7b4-41f0-8d75-0f3cff6869c0"
+				(path "/872055d3-e01a-4a82-8c05-28c93674a700/1854cea8-bf87-4849-94dd-b39855f3ac8d"
 					(reference "U7")
 					(unit 1)
@@
 			(effects (font (size 1.27 1.27)) (justify left))
 		)
-		(property "Footprint" ""
+		(property "Footprint" "Capacitor_SMD:C_1210_3225Metric"
 			(at 90.17 139.7 0)
 			(hide yes)
@@
 		(instances
 			(project "Flashover"
-				(path "/d341370c-bf24-48b8-b9fb-db9600491445/d807c62d-c7b4-41f0-8d75-0f3cff6869c0"
+				(path "/872055d3-e01a-4a82-8c05-28c93674a700/1854cea8-bf87-4849-94dd-b39855f3ac8d"
 					(reference "C3")
 					(unit 1)
@@
 		(instances
 			(project "Flashover"
-				(path "/d341370c-bf24-48b8-b9fb-db9600491445/d807c62d-c7b4-41f0-8d75-0f3cff6869c0"
+				(path "/872055d3-e01a-4a82-8c05-28c93674a700/1854cea8-bf87-4849-94dd-b39855f3ac8d"
 					(reference "#PWR06")
 					(unit 1)
@@
 			(effects (font (size 1.27 1.27)) (justify left))
 		)
-		(property "Footprint" ""
+		(property "Footprint" "Capacitor_SMD:C_0805_2012Metric"
 			(at 137.16 124.46 0)
 			(hide yes)
@@
 		(instances
 			(project "Flashover"
-				(path "/d341370c-bf24-48b8-b9fb-db9600491445/d807c62d-c7b4-41f0-8d75-0f3cff6869c0"
+				(path "/872055d3-e01a-4a82-8c05-28c93674a700/1854cea8-bf87-4849-94dd-b39855f3ac8d"
 					(reference "C10")
 					(unit 1)
@@
 		(instances
 			(project "Flashover"
-				(path "/d341370c-bf24-48b8-b9fb-db9600491445/d807c62d-c7b4-41f0-8d75-0f3cff6869c0"
+				(path "/872055d3-e01a-4a82-8c05-28c93674a700/1854cea8-bf87-4849-94dd-b39855f3ac8d"
 					(reference "#PWR07")
 					(unit 1)
@@
 		(instances
 			(project "Flashover"
-				(path "/d341370c-bf24-48b8-b9fb-db9600491445/d807c62d-c7b4-41f0-8d75-0f3cff6869c0"
+				(path "/872055d3-e01a-4a82-8c05-28c93674a700/1854cea8-bf87-4849-94dd-b39855f3ac8d"
 					(reference "#PWR08")
 					(unit 1)
