File: pedals/distortion/kicad/Flashover/midi.kicad_sch (KiCad schematic)
At the start: 9 parts, among them J5 MIDI In, J6 MIDI Out, U11 H11L1

Commit message: Apply datasheet checks to Flashover
R33 = 15k (about 5 mA per LED, from the IS31FL3236A current formula).
R39 marked 33 ohm 0.5W per MIDI CA-033. R4 390 -> 330 because the
MCP45HV51 wiper resistance is about 150 ohms at 9V (below its 10V
specified range); sim model Rw updated to match. Pot symbol description
corrected to 8-bit. Product document records the check results.

Co-Authored-By: Claude Opus 5.5 <noreply@anthropic.com>
Parts:
- R39: value 33 -> 33 0.5W
Changed lines of the file:
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@@
 		(instances
 			(project "Flashover"
-				(path "/d44d1406-41c8-4e08-862e-64ff4a05b8dc/5461588f-5b25-4dc9-ad46-4053dcc88431"
+				(path "/d341370c-bf24-48b8-b9fb-db9600491445/2c9ef750-8dcf-4430-97b2-e9f9d07dbf1c"
 					(reference "J5")
 					(unit 1)
@@
 		(instances
 			(project "Flashover"
-				(path "/d44d1406-41c8-4e08-862e-64ff4a05b8dc/5461588f-5b25-4dc9-ad46-4053dcc88431"
+				(path "/d341370c-bf24-48b8-b9fb-db9600491445/2c9ef750-8dcf-4430-97b2-e9f9d07dbf1c"
 					(reference "R37")
 					(unit 1)
@@
 		(instances
 			(project "Flashover"
-				(path "/d44d1406-41c8-4e08-862e-64ff4a05b8dc/5461588f-5b25-4dc9-ad46-4053dcc88431"
+				(path "/d341370c-bf24-48b8-b9fb-db9600491445/2c9ef750-8dcf-4430-97b2-e9f9d07dbf1c"
 					(reference "U11")
 					(unit 1)
@@
 		(instances
 			(project "Flashover"
-				(path "/d44d1406-41c8-4e08-862e-64ff4a05b8dc/5461588f-5b25-4dc9-ad46-4053dcc88431"
+				(path "/d341370c-bf24-48b8-b9fb-db9600491445/2c9ef750-8dcf-4430-97b2-e9f9d07dbf1c"
 					(reference "D43")
 					(unit 1)
@@
 		(instances
 			(project "Flashover"
-				(path "/d44d1406-41c8-4e08-862e-64ff4a05b8dc/5461588f-5b25-4dc9-ad46-4053dcc88431"
+				(path "/d341370c-bf24-48b8-b9fb-db9600491445/2c9ef750-8dcf-4430-97b2-e9f9d07dbf1c"
 					(reference "#PWR116")
 					(unit 1)
@@
 		(instances
 			(project "Flashover"
-				(path "/d44d1406-41c8-4e08-862e-64ff4a05b8dc/5461588f-5b25-4dc9-ad46-4053dcc88431"
+				(path "/d341370c-bf24-48b8-b9fb-db9600491445/2c9ef750-8dcf-4430-97b2-e9f9d07dbf1c"
 					(reference "C41")
 					(unit 1)
@@
 		(instances
 			(project "Flashover"
-				(path "/d44d1406-41c8-4e08-862e-64ff4a05b8dc/5461588f-5b25-4dc9-ad46-4053dcc88431"
+				(path "/d341370c-bf24-48b8-b9fb-db9600491445/2c9ef750-8dcf-4430-97b2-e9f9d07dbf1c"
 					(reference "#PWR117")
 					(unit 1)
@@
 		(instances
 			(project "Flashover"
-				(path "/d44d1406-41c8-4e08-862e-64ff4a05b8dc/5461588f-5b25-4dc9-ad46-4053dcc88431"
+				(path "/d341370c-bf24-48b8-b9fb-db9600491445/2c9ef750-8dcf-4430-97b2-e9f9d07dbf1c"
 					(reference "#PWR118")
 					(unit 1)
@@
 		(instances
 			(project "Flashover"
-				(path "/d44d1406-41c8-4e08-862e-64ff4a05b8dc/5461588f-5b25-4dc9-ad46-4053dcc88431"
+				(path "/d341370c-bf24-48b8-b9fb-db9600491445/2c9ef750-8dcf-4430-97b2-e9f9d07dbf1c"
 					(reference "R38")
 					(unit 1)
@@
 		(instances
 			(project "Flashover"
-				(path "/d44d1406-41c8-4e08-862e-64ff4a05b8dc/5461588f-5b25-4dc9-ad46-4053dcc88431"
+				(path "/d341370c-bf24-48b8-b9fb-db9600491445/2c9ef750-8dcf-4430-97b2-e9f9d07dbf1c"
 					(reference "#PWR119")
 					(unit 1)
@@
 		(instances
 			(project "Flashover"
-				(path "/d44d1406-41c8-4e08-862e-64ff4a05b8dc/5461588f-5b25-4dc9-ad46-4053dcc88431"
+				(path "/d341370c-bf24-48b8-b9fb-db9600491445/2c9ef750-8dcf-4430-97b2-e9f9d07dbf1c"
 					(reference "J6")
 					(unit 1)
@@
 		(instances
 			(project "Flashover"
-				(path "/d44d1406-41c8-4e08-862e-64ff4a05b8dc/5461588f-5b25-4dc9-ad46-4053dcc88431"
+				(path "/d341370c-bf24-48b8-b9fb-db9600491445/2c9ef750-8dcf-4430-97b2-e9f9d07dbf1c"
 					(reference "R40")
 					(unit 1)
@@
 			(effects (font (size 1.27 1.27)) (justify right))
 		)
-		(property "Value" "33"
+		(property "Value" "33 0.5W"
 			(at 109.22 144.78 0)
 			(show_name no)
@@
 		(instances
 			(project "Flashover"
-				(path "/d44d1406-41c8-4e08-862e-64ff4a05b8dc/5461588f-5b25-4dc9-ad46-4053dcc88431"
+				(path "/d341370c-bf24-48b8-b9fb-db9600491445/2c9ef750-8dcf-4430-97b2-e9f9d07dbf1c"
 					(reference "R39")
 					(unit 1)
@@
 		(instances
 			(project "Flashover"
-				(path "/d44d1406-41c8-4e08-862e-64ff4a05b8dc/5461588f-5b25-4dc9-ad46-4053dcc88431"
+				(path "/d341370c-bf24-48b8-b9fb-db9600491445/2c9ef750-8dcf-4430-97b2-e9f9d07dbf1c"
 					(reference "#PWR120")
 					(unit 1)
@@
 		(instances
 			(project "Flashover"
-				(path "/d44d1406-41c8-4e08-862e-64ff4a05b8dc/5461588f-5b25-4dc9-ad46-4053dcc88431"
+				(path "/d341370c-bf24-48b8-b9fb-db9600491445/2c9ef750-8dcf-4430-97b2-e9f9d07dbf1c"
 					(reference "#PWR121")
 					(unit 1)

Commit message: Assign Flashover footprints
Surface-mount for assembly; through-hole for jacks, encoders, panel LEDs,
the Soft/Hard button, the TO-220 regulator and the germanium diodes.
Q1/Q2 use the MMBT3904 symbol, 1N4148 -> 1N4148W, 1N5817 -> SS14.

Co-Authored-By: Claude Opus 5.5 <noreply@anthropic.com>
Parts:
- C41: footprint (none) -> Capacitor_SMD:C_0805_2012Metric
- D43: value 1N4148 -> 1N4148W; footprint (none) -> Diode_SMD:D_SOD-123
- J5, J6: footprint (none) -> Connector_Audio:Jack_3.5mm_CUI_SJ1-3523N_Horizontal
- R37, R38, R40: footprint (none) -> Resistor_SMD:R_0805_2012Metric
- R39: footprint (none) -> Resistor_SMD:R_2010_5025Metric
- U11: footprint (none) -> Package_DIP:SMDIP-6_W7.62mm
Changed lines of the file:
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@@
 			(effects (font (size 1.27 1.27)))
 		)
-		(property "Footprint" ""
+		(property "Footprint" "Connector_Audio:Jack_3.5mm_CUI_SJ1-3523N_Horizontal"
 			(at 30.48 83.82 0)
 			(hide yes)
@@
 		(instances
 			(project "Flashover"
-				(path "/d341370c-bf24-48b8-b9fb-db9600491445/2c9ef750-8dcf-4430-97b2-e9f9d07dbf1c"
+				(path "/872055d3-e01a-4a82-8c05-28c93674a700/a4974728-33cf-4a7c-98bf-cb86e0234eaf"
 					(reference "J5")
 					(unit 1)
@@
 			(effects (font (size 1.27 1.27)))
 		)
-		(property "Footprint" ""
+		(property "Footprint" "Resistor_SMD:R_0805_2012Metric"
 			(at 48.26 83.82 90)
 			(hide yes)
@@
 		(instances
 			(project "Flashover"
-				(path "/d341370c-bf24-48b8-b9fb-db9600491445/2c9ef750-8dcf-4430-97b2-e9f9d07dbf1c"
+				(path "/872055d3-e01a-4a82-8c05-28c93674a700/a4974728-33cf-4a7c-98bf-cb86e0234eaf"
 					(reference "R37")
 					(unit 1)
@@
 			(effects (font (size 1.27 1.27)))
 		)
-		(property "Footprint" ""
+		(property "Footprint" "Package_DIP:SMDIP-6_W7.62mm"
 			(at 86.36 86.36 0)
 			(hide yes)
@@
 		(instances
 			(project "Flashover"
-				(path "/d341370c-bf24-48b8-b9fb-db9600491445/2c9ef750-8dcf-4430-97b2-e9f9d07dbf1c"
+				(path "/872055d3-e01a-4a82-8c05-28c93674a700/a4974728-33cf-4a7c-98bf-cb86e0234eaf"
 					(reference "U11")
 					(unit 1)
@@
 			(effects (font (size 1.27 1.27)))
 		)
-		(property "Value" "1N4148"
-			(at 57.531 88.9 270)
-			(show_name no)
-			(do_not_autoplace no)
-			(effects (font (size 1.27 1.27)))
-		)
-		(property "Footprint" ""
+		(property "Value" "1N4148W"
+			(at 56.9595 88.9 270)
+			(show_name no)
+			(do_not_autoplace no)
+			(effects (font (size 1.27 1.27)))
+		)
+		(property "Footprint" "Diode_SMD:D_SOD-123"
 			(at 63.5 87.63 270)
 			(hide yes)
@@
 		(instances
 			(project "Flashover"
-				(path "/d341370c-bf24-48b8-b9fb-db9600491445/2c9ef750-8dcf-4430-97b2-e9f9d07dbf1c"
+				(path "/872055d3-e01a-4a82-8c05-28c93674a700/a4974728-33cf-4a7c-98bf-cb86e0234eaf"
 					(reference "D43")
 					(unit 1)
@@
 		(instances
 			(project "Flashover"
-				(path "/d341370c-bf24-48b8-b9fb-db9600491445/2c9ef750-8dcf-4430-97b2-e9f9d07dbf1c"
+				(path "/872055d3-e01a-4a82-8c05-28c93674a700/a4974728-33cf-4a7c-98bf-cb86e0234eaf"
 					(reference "#PWR116")
 					(unit 1)
@@
 			(effects (font (size 1.27 1.27)) (justify right))
 		)
-		(property "Footprint" ""
+		(property "Footprint" "Capacitor_SMD:C_0805_2012Metric"
 			(at 99.06 77.47 0)
 			(hide yes)
@@
 		(instances
 			(project "Flashover"
-				(path "/d341370c-bf24-48b8-b9fb-db9600491445/2c9ef750-8dcf-4430-97b2-e9f9d07dbf1c"
+				(path "/872055d3-e01a-4a82-8c05-28c93674a700/a4974728-33cf-4a7c-98bf-cb86e0234eaf"
 					(reference "C41")
 					(unit 1)
@@
 		(instances
 			(project "Flashover"
-				(path "/d341370c-bf24-48b8-b9fb-db9600491445/2c9ef750-8dcf-4430-97b2-e9f9d07dbf1c"
+				(path "/872055d3-e01a-4a82-8c05-28c93674a700/a4974728-33cf-4a7c-98bf-cb86e0234eaf"
 					(reference "#PWR117")
 					(unit 1)
@@
 		(instances
 			(project "Flashover"
-				(path "/d341370c-bf24-48b8-b9fb-db9600491445/2c9ef750-8dcf-4430-97b2-e9f9d07dbf1c"
+				(path "/872055d3-e01a-4a82-8c05-28c93674a700/a4974728-33cf-4a7c-98bf-cb86e0234eaf"
 					(reference "#PWR118")
 					(unit 1)
@@
 			(effects (font (size 1.27 1.27)) (justify left))
 		)
-		(property "Footprint" ""
+		(property "Footprint" "Resistor_SMD:R_0805_2012Metric"
 			(at 106.68 82.55 0)
 			(hide yes)
@@
 		(instances
 			(project "Flashover"
-				(path "/d341370c-bf24-48b8-b9fb-db9600491445/2c9ef750-8dcf-4430-97b2-e9f9d07dbf1c"
+				(path "/872055d3-e01a-4a82-8c05-28c93674a700/a4974728-33cf-4a7c-98bf-cb86e0234eaf"
 					(reference "R38")
 					(unit 1)
@@
 		(instances
 			(project "Flashover"
-				(path "/d341370c-bf24-48b8-b9fb-db9600491445/2c9ef750-8dcf-4430-97b2-e9f9d07dbf1c"
+				(path "/872055d3-e01a-4a82-8c05-28c93674a700/a4974728-33cf-4a7c-98bf-cb86e0234eaf"
 					(reference "#PWR119")
 					(unit 1)
@@
 			(effects (font (size 1.27 1.27)))
 		)
-		(property "Footprint" ""
+		(property "Footprint" "Connector_Audio:Jack_3.5mm_CUI_SJ1-3523N_Horizontal"
 			(at 124.46 139.7 0)
 			(hide yes)
@@
 		(instances
 			(project "Flashover"
-				(path "/d341370c-bf24-48b8-b9fb-db9600491445/2c9ef750-8dcf-4430-97b2-e9f9d07dbf1c"
+				(path "/872055d3-e01a-4a82-8c05-28c93674a700/a4974728-33cf-4a7c-98bf-cb86e0234eaf"
 					(reference "J6")
 					(unit 1)
@@
 			(effects (font (size 1.27 1.27)))
 		)
-		(property "Footprint" ""
+		(property "Footprint" "Resistor_SMD:R_0805_2012Metric"
 			(at 104.14 137.16 90)
 			(hide yes)
@@
 		(instances
 			(project "Flashover"
-				(path "/d341370c-bf24-48b8-b9fb-db9600491445/2c9ef750-8dcf-4430-97b2-e9f9d07dbf1c"
+				(path "/872055d3-e01a-4a82-8c05-28c93674a700/a4974728-33cf-4a7c-98bf-cb86e0234eaf"
 					(reference "R40")
 					(unit 1)
@@
 			(effects (font (size 1.27 1.27)) (justify right))
 		)
-		(property "Footprint" ""
+		(property "Footprint" "Resistor_SMD:R_2010_5025Metric"
 			(at 111.76 143.51 0)
 			(hide yes)
@@
 		(instances
 			(project "Flashover"
-				(path "/d341370c-bf24-48b8-b9fb-db9600491445/2c9ef750-8dcf-4430-97b2-e9f9d07dbf1c"
+				(path "/872055d3-e01a-4a82-8c05-28c93674a700/a4974728-33cf-4a7c-98bf-cb86e0234eaf"
 					(reference "R39")
 					(unit 1)
@@
 		(instances
 			(project "Flashover"
-				(path "/d341370c-bf24-48b8-b9fb-db9600491445/2c9ef750-8dcf-4430-97b2-e9f9d07dbf1c"
+				(path "/872055d3-e01a-4a82-8c05-28c93674a700/a4974728-33cf-4a7c-98bf-cb86e0234eaf"
 					(reference "#PWR120")
 					(unit 1)
@@
 		(instances
 			(project "Flashover"
-				(path "/d341370c-bf24-48b8-b9fb-db9600491445/2c9ef750-8dcf-4430-97b2-e9f9d07dbf1c"
+				(path "/872055d3-e01a-4a82-8c05-28c93674a700/a4974728-33cf-4a7c-98bf-cb86e0234eaf"
 					(reference "#PWR121")
 					(unit 1)
