File: pedals/distortion/kicad/Flashover/tone_output.kicad_sch (KiCad schematic)
At the start: 12 parts, among them J2 Output, U2 TL072

Commit message: Add Flashover controller and digital pot sheets
Controller sheet: RP2040 with 3.3V regulator, 2 MB QSPI flash, 12 MHz
crystal and SWD header, plus a GPIO plan for the sheets still to come.
Digital Pots sheet: control side of three MCP45HV51 I2C pots with
pull-ups. RV1-RV3 on the audio sheets become the pot units of U7-U9
(new two-unit MCP45HV51 symbol in the shared library). ERC clean.

Co-Authored-By: Claude Opus 5.5 <noreply@anthropic.com>
Parts:
- removed RV2, RV3: 10k digital, symbol Device:R_Potentiometer
- added U8, U9: MCP45HV51-103, symbol GreywireStudio:MCP45HV51
Connections:
- net VB: now also U9.11
- net at R16.2, U2.1: now also U9.13
- net at U2.3 (+): now also U8.12
- net at C8.2, R14.2: now also U8.13
- net at C9.1: now also U9.12
- net at C12.2, R15.1: now also U8.11
Other:
- note added: "U8A (Tone) and U9A (Level) are MCP45HV51 digital pots (10k); their control and power pins are on the Digital Pots sheet. Everything after the gain stage is centered on VB (4.5V) so the digital pots only see 0V to 9V. Level is reduced to about 38% in Hard mode to match Soft's volume."
- note removed: "RV2 (Tone) and RV3 (Level) are MCP41HV digital pots. Everything after the gain stage is centered on VB (4.5V) so the digital pots only see 0V to 9V. Level is reduced to about 38% in Hard mode to match Soft's volume."
Changed lines of the file:
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@@
 	(rectangle
 		(start 68.58 53.34)
-		(end 121.92 124.46)
+		(end 116.84 124.46)
 		(stroke (width 0) (type dash))
 		(fill (type none))
@@
 	)
 	(rectangle
-		(start 121.92 53.34)
+		(start 116.84 53.34)
 		(end 185.42 124.46)
 		(stroke (width 0) (type dash))
@@
 	(text "G: LEVEL AND OUTPUT"
 		(exclude_from_sim no)
-		(at 123.19 55.245 0)
+		(at 118.11 55.245 0)
 		(effects (font (size 1.524 1.524) (bold yes)) (justify left))
 	)
@@
 		(effects (font (size 1 1)) (justify left))
 	)
-	(text "RV2 (Tone) and RV3 (Level) are MCP41HV digital pots.\nEverything after the gain stage is centered on VB (4.5V)\nso the digital pots only see 0V to 9V.\nLevel is reduced to about 38% in Hard mode to match Soft's volume."
+	(text "U8A (Tone) and U9A (Level) are MCP45HV51 digital pots (10k);\ntheir control and power pins are on the Digital Pots sheet.\nEverything after the gain stage is centered on VB (4.5V)\nso the digital pots only see 0V to 9V.\nLevel is reduced to about 38% in Hard mode to match Soft's volume."
 		(exclude_from_sim no)
 		(at 20.32 134.62 0)
@@
 		(instances
 			(project "Flashover"
-				(path "/c1c20152-b132-4e14-97dc-1ac24480e45d/c612ce62-484a-452b-bbb9-31deb194e553"
+				(path "/37bda491-c0dc-4d48-acdf-49df4f139bb0/641032a7-af45-463f-9bff-064e3d76b912"
 					(reference "R14")
 					(unit 1)
@@
 		(instances
 			(project "Flashover"
-				(path "/c1c20152-b132-4e14-97dc-1ac24480e45d/c612ce62-484a-452b-bbb9-31deb194e553"
+				(path "/37bda491-c0dc-4d48-acdf-49df4f139bb0/641032a7-af45-463f-9bff-064e3d76b912"
 					(reference "C12")
 					(unit 1)
@@
 		(instances
 			(project "Flashover"
-				(path "/c1c20152-b132-4e14-97dc-1ac24480e45d/c612ce62-484a-452b-bbb9-31deb194e553"
+				(path "/37bda491-c0dc-4d48-acdf-49df4f139bb0/641032a7-af45-463f-9bff-064e3d76b912"
 					(reference "C8")
 					(unit 1)
@@
 		(instances
 			(project "Flashover"
-				(path "/c1c20152-b132-4e14-97dc-1ac24480e45d/c612ce62-484a-452b-bbb9-31deb194e553"
+				(path "/37bda491-c0dc-4d48-acdf-49df4f139bb0/641032a7-af45-463f-9bff-064e3d76b912"
 					(reference "#PWR17")
 					(unit 1)
@@
 		(instances
 			(project "Flashover"
-				(path "/c1c20152-b132-4e14-97dc-1ac24480e45d/c612ce62-484a-452b-bbb9-31deb194e553"
+				(path "/37bda491-c0dc-4d48-acdf-49df4f139bb0/641032a7-af45-463f-9bff-064e3d76b912"
 					(reference "R15")
 					(unit 1)
@@
 		(instances
 			(project "Flashover"
-				(path "/c1c20152-b132-4e14-97dc-1ac24480e45d/c612ce62-484a-452b-bbb9-31deb194e553"
+				(path "/37bda491-c0dc-4d48-acdf-49df4f139bb0/641032a7-af45-463f-9bff-064e3d76b912"
 					(reference "#PWR18")
 					(unit 1)
@@
 	)
 	(symbol
-		(lib_id "Device:R_Potentiometer")
+		(lib_id "GreywireStudio:MCP45HV51")
 		(at 60.96 83.82 0)
 		(unit 1)
@@
 		(in_pos_files yes)
 		(dnp no)
-		(property "Reference" "RV2"
-			(at 63.5 76.2 0)
-			(show_name no)
-			(do_not_autoplace no)
-			(effects (font (size 1.27 1.27)) (justify left))
-		)
-		(property "Value" "10k digital"
-			(at 63.5 78.105 0)
-			(show_name no)
-			(do_not_autoplace no)
-			(effects (font (size 1.27 1.27)) (justify left))
+		(property "Reference" "U8"
+			(at 58.42 82.55 0)
+			(show_name no)
+			(do_not_autoplace no)
+			(effects (font (size 1.27 1.27)) (justify right))
+		)
+		(property "Value" "MCP45HV51-103"
+			(at 58.42 85.09 0)
+			(show_name no)
+			(do_not_autoplace no)
+			(effects (font (size 1.27 1.27)) (justify right))
 		)
 		(property "Footprint" ""
@@
 			(effects (font (size 1.27 1.27)))
 		)
-		(pin "1"
-		)
-		(pin "2"
-		)
-		(pin "3"
-		)
-		(instances
-			(project "Flashover"
-				(path "/c1c20152-b132-4e14-97dc-1ac24480e45d/c612ce62-484a-452b-bbb9-31deb194e553"
-					(reference "RV2")
+		(pin "13"
+		)
+		(pin "12"
+		)
+		(pin "11"
+		)
+		(instances
+			(project "Flashover"
+				(path "/37bda491-c0dc-4d48-acdf-49df4f139bb0/641032a7-af45-463f-9bff-064e3d76b912"
+					(reference "U8")
 					(unit 1)
 				)
@@
 		(instances
 			(project "Flashover"
-				(path "/c1c20152-b132-4e14-97dc-1ac24480e45d/c612ce62-484a-452b-bbb9-31deb194e553"
+				(path "/37bda491-c0dc-4d48-acdf-49df4f139bb0/641032a7-af45-463f-9bff-064e3d76b912"
 					(reference "U2")
 					(unit 1)
@@
 		(instances
 			(project "Flashover"
-				(path "/c1c20152-b132-4e14-97dc-1ac24480e45d/c612ce62-484a-452b-bbb9-31deb194e553"
+				(path "/37bda491-c0dc-4d48-acdf-49df4f139bb0/641032a7-af45-463f-9bff-064e3d76b912"
 					(reference "R16")
 					(unit 1)
@@
 		(instances
 			(project "Flashover"
-				(path "/c1c20152-b132-4e14-97dc-1ac24480e45d/c612ce62-484a-452b-bbb9-31deb194e553"
+				(path "/37bda491-c0dc-4d48-acdf-49df4f139bb0/641032a7-af45-463f-9bff-064e3d76b912"
 					(reference "R17")
 					(unit 1)
@@
 		(instances
 			(project "Flashover"
-				(path "/c1c20152-b132-4e14-97dc-1ac24480e45d/c612ce62-484a-452b-bbb9-31deb194e553"
+				(path "/37bda491-c0dc-4d48-acdf-49df4f139bb0/641032a7-af45-463f-9bff-064e3d76b912"
 					(reference "#PWR19")
 					(unit 1)
@@
 	)
 	(symbol
-		(lib_id "Device:R_Potentiometer")
+		(lib_id "GreywireStudio:MCP45HV51")
 		(at 137.16 93.98 0)
 		(unit 1)
@@
 		(in_pos_files yes)
 		(dnp no)
-		(property "Reference" "RV3"
+		(property "Reference" "U9"
 			(at 134.62 92.71 0)
 			(show_name no)
@@
 			(effects (font (size 1.27 1.27)) (justify right))
 		)
-		(property "Value" "10k digital"
+		(property "Value" "MCP45HV51-103"
 			(at 134.62 95.25 0)
 			(show_name no)
@@
 			(effects (font (size 1.27 1.27)))
 		)
-		(pin "1"
-		)
-		(pin "2"
-		)
-		(pin "3"
-		)
-		(instances
-			(project "Flashover"
-				(path "/c1c20152-b132-4e14-97dc-1ac24480e45d/c612ce62-484a-452b-bbb9-31deb194e553"
-					(reference "RV3")
+		(pin "13"
+		)
+		(pin "12"
+		)
+		(pin "11"
+		)
+		(instances
+			(project "Flashover"
+				(path "/37bda491-c0dc-4d48-acdf-49df4f139bb0/641032a7-af45-463f-9bff-064e3d76b912"
+					(reference "U9")
 					(unit 1)
 				)
@@
 		(instances
 			(project "Flashover"
-				(path "/c1c20152-b132-4e14-97dc-1ac24480e45d/c612ce62-484a-452b-bbb9-31deb194e553"
+				(path "/37bda491-c0dc-4d48-acdf-49df4f139bb0/641032a7-af45-463f-9bff-064e3d76b912"
 					(reference "#PWR20")
 					(unit 1)
@@
 		(instances
 			(project "Flashover"
-				(path "/c1c20152-b132-4e14-97dc-1ac24480e45d/c612ce62-484a-452b-bbb9-31deb194e553"
+				(path "/37bda491-c0dc-4d48-acdf-49df4f139bb0/641032a7-af45-463f-9bff-064e3d76b912"
 					(reference "C9")
 					(unit 1)
@@
 		(instances
 			(project "Flashover"
-				(path "/c1c20152-b132-4e14-97dc-1ac24480e45d/c612ce62-484a-452b-bbb9-31deb194e553"
+				(path "/37bda491-c0dc-4d48-acdf-49df4f139bb0/641032a7-af45-463f-9bff-064e3d76b912"
 					(reference "R11")
 					(unit 1)
@@
 		(instances
 			(project "Flashover"
-				(path "/c1c20152-b132-4e14-97dc-1ac24480e45d/c612ce62-484a-452b-bbb9-31deb194e553"
+				(path "/37bda491-c0dc-4d48-acdf-49df4f139bb0/641032a7-af45-463f-9bff-064e3d76b912"
 					(reference "J2")
 					(unit 1)
@@
 		(instances
 			(project "Flashover"
-				(path "/c1c20152-b132-4e14-97dc-1ac24480e45d/c612ce62-484a-452b-bbb9-31deb194e553"
+				(path "/37bda491-c0dc-4d48-acdf-49df4f139bb0/641032a7-af45-463f-9bff-064e3d76b912"
 					(reference "#PWR21")
 					(unit 1)
@@
 		(instances
 			(project "Flashover"
-				(path "/c1c20152-b132-4e14-97dc-1ac24480e45d/c612ce62-484a-452b-bbb9-31deb194e553"
+				(path "/37bda491-c0dc-4d48-acdf-49df4f139bb0/641032a7-af45-463f-9bff-064e3d76b912"
 					(reference "#PWR22")
 					(unit 1)

Commit message: Add Flashover bypass sheet; complete schematic
Bypass sheet: fail-safe G6K-2 relay bypass (NC contacts join the jacks
when unpowered), input/output jacks moved here from the audio sheets
(now FX_IN/FX_OUT), relay driver on FX_ON, soft-touch footswitch and
Link LED. Relay coils on K1 and K2 now take +5V on pin 1 (marked +).
Root sheet laid out in four columns. ERC clean.

Co-Authored-By: Claude Opus 5.5 <noreply@anthropic.com>
Parts:
- removed J2: Output, symbol Connector_Audio:AudioJack2
Connections:
- net FX_OUT: now reaches C9.2, R11.1
Other:
- note added: "FX_OUT goes to the output jack through the bypass relay (Bypass sheet)."
Changed lines of the file:
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@@
 	(wire
 		(pts
-			(xy 154.94 93.98) (xy 170.18 93.98)
+			(xy 154.94 93.98) (xy 165.1 93.98)
 		)
 		(stroke
@@
 		(pts
 			(xy 154.94 93.98) (xy 154.94 99.06)
-		)
-		(stroke
-			(width 0)
-			(type default)
-		)
-	)
-	(wire
-		(pts
-			(xy 170.18 96.52) (xy 167.64 96.52)
-		)
-		(stroke
-			(width 0)
-			(type default)
-		)
-	)
-	(wire
-		(pts
-			(xy 167.64 96.52) (xy 167.64 101.6)
 		)
 		(stroke
@@
 		(effects (font (size 1 1)) (justify left))
 	)
+	(global_label "FX_OUT"
+		(shape output)
+		(at 165.1 93.98 0)
+		(fields_autoplaced yes)
+		(effects (font (size 1.27 1.27)) (justify left))
+		(property "Intersheetrefs" "${INTERSHEET_REFS}"
+			(at 165.1 93.98 0)
+			(effects (font (size 1.27 1.27)) (justify left) (hide yes))
+		)
+	)
+	(text "FX_OUT goes to the output jack\nthrough the bypass relay\n(Bypass sheet)."
+		(exclude_from_sim no)
+		(at 158.75 114.3 0)
+		(effects (font (size 1 1)) (justify left))
+	)
 	(text "Gain = 1 + R16 / R17 = 4 (+12 dB), makes up the tone network's loss"
 		(exclude_from_sim no)
@@
 		(instances
 			(project "Flashover"
-				(path "/6aa723b4-171b-4dbf-8521-b922c86d1498/f894bec3-848a-42fa-b2be-5c928a7f08b6"
+				(path "/d44d1406-41c8-4e08-862e-64ff4a05b8dc/d799564d-b3cd-4934-9403-fb4471bc03b2"
 					(reference "R14")
 					(unit 1)
@@
 		(instances
 			(project "Flashover"
-				(path "/6aa723b4-171b-4dbf-8521-b922c86d1498/f894bec3-848a-42fa-b2be-5c928a7f08b6"
+				(path "/d44d1406-41c8-4e08-862e-64ff4a05b8dc/d799564d-b3cd-4934-9403-fb4471bc03b2"
 					(reference "C12")
 					(unit 1)
@@
 		(instances
 			(project "Flashover"
-				(path "/6aa723b4-171b-4dbf-8521-b922c86d1498/f894bec3-848a-42fa-b2be-5c928a7f08b6"
+				(path "/d44d1406-41c8-4e08-862e-64ff4a05b8dc/d799564d-b3cd-4934-9403-fb4471bc03b2"
 					(reference "C8")
 					(unit 1)
@@
 		(in_pos_files yes)
 		(dnp no)
-		(property "Reference" "#PWR17"
+		(property "Reference" "#PWR16"
 			(at 50.8 67.31 0)
 			(hide yes)
@@
 		(instances
 			(project "Flashover"
-				(path "/6aa723b4-171b-4dbf-8521-b922c86d1498/f894bec3-848a-42fa-b2be-5c928a7f08b6"
-					(reference "#PWR17")
+				(path "/d44d1406-41c8-4e08-862e-64ff4a05b8dc/d799564d-b3cd-4934-9403-fb4471bc03b2"
+					(reference "#PWR16")
 					(unit 1)
 				)
@@
 		(instances
 			(project "Flashover"
-				(path "/6aa723b4-171b-4dbf-8521-b922c86d1498/f894bec3-848a-42fa-b2be-5c928a7f08b6"
+				(path "/d44d1406-41c8-4e08-862e-64ff4a05b8dc/d799564d-b3cd-4934-9403-fb4471bc03b2"
 					(reference "R15")
 					(unit 1)
@@
 		(in_pos_files yes)
 		(dnp no)
-		(property "Reference" "#PWR18"
+		(property "Reference" "#PWR17"
 			(at 50.8 110.49 0)
 			(hide yes)
@@
 		(instances
 			(project "Flashover"
-				(path "/6aa723b4-171b-4dbf-8521-b922c86d1498/f894bec3-848a-42fa-b2be-5c928a7f08b6"
-					(reference "#PWR18")
+				(path "/d44d1406-41c8-4e08-862e-64ff4a05b8dc/d799564d-b3cd-4934-9403-fb4471bc03b2"
+					(reference "#PWR17")
 					(unit 1)
 				)
@@
 		(instances
 			(project "Flashover"
-				(path "/6aa723b4-171b-4dbf-8521-b922c86d1498/f894bec3-848a-42fa-b2be-5c928a7f08b6"
+				(path "/d44d1406-41c8-4e08-862e-64ff4a05b8dc/d799564d-b3cd-4934-9403-fb4471bc03b2"
 					(reference "U8")
 					(unit 1)
@@
 		(instances
 			(project "Flashover"
-				(path "/6aa723b4-171b-4dbf-8521-b922c86d1498/f894bec3-848a-42fa-b2be-5c928a7f08b6"
+				(path "/d44d1406-41c8-4e08-862e-64ff4a05b8dc/d799564d-b3cd-4934-9403-fb4471bc03b2"
 					(reference "U2")
 					(unit 1)
@@
 		(instances
 			(project "Flashover"
-				(path "/6aa723b4-171b-4dbf-8521-b922c86d1498/f894bec3-848a-42fa-b2be-5c928a7f08b6"
+				(path "/d44d1406-41c8-4e08-862e-64ff4a05b8dc/d799564d-b3cd-4934-9403-fb4471bc03b2"
 					(reference "R16")
 					(unit 1)
@@
 		(instances
 			(project "Flashover"
-				(path "/6aa723b4-171b-4dbf-8521-b922c86d1498/f894bec3-848a-42fa-b2be-5c928a7f08b6"
+				(path "/d44d1406-41c8-4e08-862e-64ff4a05b8dc/d799564d-b3cd-4934-9403-fb4471bc03b2"
 					(reference "R17")
 					(unit 1)
@@
 		(in_pos_files yes)
 		(dnp no)
-		(property "Reference" "#PWR19"
+		(property "Reference" "#PWR18"
 			(at 71.12 116.84 0)
 			(hide yes)
@@
 		(instances
 			(project "Flashover"
-				(path "/6aa723b4-171b-4dbf-8521-b922c86d1498/f894bec3-848a-42fa-b2be-5c928a7f08b6"
-					(reference "#PWR19")
+				(path "/d44d1406-41c8-4e08-862e-64ff4a05b8dc/d799564d-b3cd-4934-9403-fb4471bc03b2"
+					(reference "#PWR18")
 					(unit 1)
 				)
@@
 		(instances
 			(project "Flashover"
-				(path "/6aa723b4-171b-4dbf-8521-b922c86d1498/f894bec3-848a-42fa-b2be-5c928a7f08b6"
+				(path "/d44d1406-41c8-4e08-862e-64ff4a05b8dc/d799564d-b3cd-4934-9403-fb4471bc03b2"
 					(reference "U9")
 					(unit 1)
@@
 		(in_pos_files yes)
 		(dnp no)
-		(property "Reference" "#PWR20"
+		(property "Reference" "#PWR19"
 			(at 137.16 104.14 0)
 			(hide yes)
@@
 		(instances
 			(project "Flashover"
-				(path "/6aa723b4-171b-4dbf-8521-b922c86d1498/f894bec3-848a-42fa-b2be-5c928a7f08b6"
-					(reference "#PWR20")
+				(path "/d44d1406-41c8-4e08-862e-64ff4a05b8dc/d799564d-b3cd-4934-9403-fb4471bc03b2"
+					(reference "#PWR19")
 					(unit 1)
 				)
@@
 		(instances
 			(project "Flashover"
-				(path "/6aa723b4-171b-4dbf-8521-b922c86d1498/f894bec3-848a-42fa-b2be-5c928a7f08b6"
+				(path "/d44d1406-41c8-4e08-862e-64ff4a05b8dc/d799564d-b3cd-4934-9403-fb4471bc03b2"
 					(reference "C9")
 					(unit 1)
@@
 		(instances
 			(project "Flashover"
-				(path "/6aa723b4-171b-4dbf-8521-b922c86d1498/f894bec3-848a-42fa-b2be-5c928a7f08b6"
+				(path "/d44d1406-41c8-4e08-862e-64ff4a05b8dc/d799564d-b3cd-4934-9403-fb4471bc03b2"
 					(reference "R11")
-					(unit 1)
-				)
-			)
-		)
-	)
-	(symbol
-		(lib_id "Connector_Audio:AudioJack2")
-		(at 175.26 93.98 180)
-		(unit 1)
-		(body_style 1)
-		(exclude_from_sim no)
-		(in_bom yes)
-		(on_board yes)
-		(in_pos_files yes)
-		(dnp no)
-		(property "Reference" "J2"
-			(at 177.8 86.36 0)
-			(show_name no)
-			(do_not_autoplace no)
-			(effects (font (size 1.27 1.27)))
-		)
-		(property "Value" "Output"
-			(at 177.8 88.9 0)
-			(show_name no)
-			(do_not_autoplace no)
-			(effects (font (size 1.27 1.27)))
-		)
-		(property "Footprint" ""
-			(at 175.26 93.98 0)
-			(hide yes)
-			(show_name no)
-			(do_not_autoplace no)
-			(effects (font (size 1.27 1.27)))
-		)
-		(property "Datasheet" ""
-			(at 175.26 93.98 0)
-			(hide yes)
-			(show_name no)
-			(do_not_autoplace no)
-			(effects (font (size 1.27 1.27)))
-		)
-		(pin "S"
-		)
-		(pin "T"
-		)
-		(instances
-			(project "Flashover"
-				(path "/6aa723b4-171b-4dbf-8521-b922c86d1498/f894bec3-848a-42fa-b2be-5c928a7f08b6"
-					(reference "J2")
 					(unit 1)
 				)
@@
 		(in_pos_files yes)
 		(dnp no)
-		(property "Reference" "#PWR21"
+		(property "Reference" "#PWR20"
 			(at 154.94 113.03 0)
 			(hide yes)
@@
 		(instances
 			(project "Flashover"
-				(path "/6aa723b4-171b-4dbf-8521-b922c86d1498/f894bec3-848a-42fa-b2be-5c928a7f08b6"
-					(reference "#PWR21")
-					(unit 1)
-				)
-			)
-		)
-	)
-	(symbol
-		(lib_id "power:GND")
-		(at 167.64 101.6 0)
-		(unit 1)
-		(body_style 1)
-		(exclude_from_sim no)
-		(in_bom no)
-		(on_board no)
-		(in_pos_files yes)
-		(dnp no)
-		(property "Reference" "#PWR22"
-			(at 167.64 107.95 0)
-			(hide yes)
-			(show_name no)
-			(do_not_autoplace no)
-			(effects (font (size 1.27 1.27)))
-		)
-		(property "Value" "GND"
-			(at 167.64 105.41 0)
-			(show_name no)
-			(do_not_autoplace no)
-			(effects (font (size 1.27 1.27)))
-		)
-		(property "Footprint" ""
-			(at 167.64 101.6 0)
-			(hide yes)
-			(show_name no)
-			(do_not_autoplace no)
-			(effects (font (size 1.27 1.27)))
-		)
-		(property "Datasheet" ""
-			(at 167.64 101.6 0)
-			(hide yes)
-			(show_name no)
-			(do_not_autoplace no)
-			(effects (font (size 1.27 1.27)))
-		)
-		(pin "1"
-		)
-		(instances
-			(project "Flashover"
-				(path "/6aa723b4-171b-4dbf-8521-b922c86d1498/f894bec3-848a-42fa-b2be-5c928a7f08b6"
-					(reference "#PWR22")
-					(unit 1)
-				)
+				(path "/d44d1406-41c8-4e08-862e-64ff4a05b8dc/d799564d-b3cd-4934-9403-fb4471bc03b2"
+					(reference "#PWR20")
+					(unit 1)
+				)
