File: pedals/distortion/kicad/Flashover/tone_output.kicad_sch (KiCad schematic)
At the start: 11 parts, among them U2 TL072, U8 MCP45HV51-103, U9 MCP45HV51-103

Commit message: Assign Flashover footprints
Surface-mount for assembly; through-hole for jacks, encoders, panel LEDs,
the Soft/Hard button, the TO-220 regulator and the germanium diodes.
Q1/Q2 use the MMBT3904 symbol, 1N4148 -> 1N4148W, 1N5817 -> SS14.

Co-Authored-By: Claude Opus 5.5 <noreply@anthropic.com>
Parts:
- C12, C8: footprint (none) -> Capacitor_SMD:C_1206_3216Metric
- C9: footprint (none) -> Capacitor_SMD:C_1210_3225Metric
- R11, R14, R15, R16, R17: footprint (none) -> Resistor_SMD:R_0805_2012Metric
- U2: footprint (none) -> Package_SO:SOIC-8_3.9x4.9mm_P1.27mm
- U8, U9: footprint (none) -> Package_SO:TSSOP-14_4.4x5mm_P0.65mm
Changed lines of the file:
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@@
 			(effects (font (size 1.27 1.27)))
 		)
-		(property "Footprint" ""
+		(property "Footprint" "Resistor_SMD:R_0805_2012Metric"
 			(at 40.64 76.2 90)
 			(hide yes)
@@
 		(instances
 			(project "Flashover"
-				(path "/d341370c-bf24-48b8-b9fb-db9600491445/b4d4908f-d3cb-45c8-9e34-8e6e14bfce1f"
+				(path "/872055d3-e01a-4a82-8c05-28c93674a700/e0ce4150-4c2b-4816-bb42-05bac40058e5"
 					(reference "R14")
 					(unit 1)
@@
 			(effects (font (size 1.27 1.27)))
 		)
-		(property "Footprint" ""
+		(property "Footprint" "Capacitor_SMD:C_1206_3216Metric"
 			(at 40.64 91.44 90)
 			(hide yes)
@@
 		(instances
 			(project "Flashover"
-				(path "/d341370c-bf24-48b8-b9fb-db9600491445/b4d4908f-d3cb-45c8-9e34-8e6e14bfce1f"
+				(path "/872055d3-e01a-4a82-8c05-28c93674a700/e0ce4150-4c2b-4816-bb42-05bac40058e5"
 					(reference "C12")
 					(unit 1)
@@
 			(effects (font (size 1.27 1.27)) (justify left))
 		)
-		(property "Footprint" ""
+		(property "Footprint" "Capacitor_SMD:C_1206_3216Metric"
 			(at 50.8 67.31 0)
 			(hide yes)
@@
 		(instances
 			(project "Flashover"
-				(path "/d341370c-bf24-48b8-b9fb-db9600491445/b4d4908f-d3cb-45c8-9e34-8e6e14bfce1f"
+				(path "/872055d3-e01a-4a82-8c05-28c93674a700/e0ce4150-4c2b-4816-bb42-05bac40058e5"
 					(reference "C8")
 					(unit 1)
@@
 		(instances
 			(project "Flashover"
-				(path "/d341370c-bf24-48b8-b9fb-db9600491445/b4d4908f-d3cb-45c8-9e34-8e6e14bfce1f"
+				(path "/872055d3-e01a-4a82-8c05-28c93674a700/e0ce4150-4c2b-4816-bb42-05bac40058e5"
 					(reference "#PWR16")
 					(unit 1)
@@
 			(effects (font (size 1.27 1.27)) (justify left))
 		)
-		(property "Footprint" ""
+		(property "Footprint" "Resistor_SMD:R_0805_2012Metric"
 			(at 50.8 100.33 0)
 			(hide yes)
@@
 		(instances
 			(project "Flashover"
-				(path "/d341370c-bf24-48b8-b9fb-db9600491445/b4d4908f-d3cb-45c8-9e34-8e6e14bfce1f"
+				(path "/872055d3-e01a-4a82-8c05-28c93674a700/e0ce4150-4c2b-4816-bb42-05bac40058e5"
 					(reference "R15")
 					(unit 1)
@@
 		(instances
 			(project "Flashover"
-				(path "/d341370c-bf24-48b8-b9fb-db9600491445/b4d4908f-d3cb-45c8-9e34-8e6e14bfce1f"
+				(path "/872055d3-e01a-4a82-8c05-28c93674a700/e0ce4150-4c2b-4816-bb42-05bac40058e5"
 					(reference "#PWR17")
 					(unit 1)
@@
 			(effects (font (size 1.27 1.27)) (justify right))
 		)
-		(property "Footprint" ""
+		(property "Footprint" "Package_SO:TSSOP-14_4.4x5mm_P0.65mm"
 			(at 60.96 83.82 0)
 			(hide yes)
@@
 		(instances
 			(project "Flashover"
-				(path "/d341370c-bf24-48b8-b9fb-db9600491445/b4d4908f-d3cb-45c8-9e34-8e6e14bfce1f"
+				(path "/872055d3-e01a-4a82-8c05-28c93674a700/e0ce4150-4c2b-4816-bb42-05bac40058e5"
 					(reference "U8")
 					(unit 1)
@@
 			(effects (font (size 1.27 1.27)) (justify left))
 		)
-		(property "Footprint" ""
+		(property "Footprint" "Package_SO:SOIC-8_3.9x4.9mm_P1.27mm"
 			(at 81.28 86.36 0)
 			(hide yes)
@@
 		(instances
 			(project "Flashover"
-				(path "/d341370c-bf24-48b8-b9fb-db9600491445/b4d4908f-d3cb-45c8-9e34-8e6e14bfce1f"
+				(path "/872055d3-e01a-4a82-8c05-28c93674a700/e0ce4150-4c2b-4816-bb42-05bac40058e5"
 					(reference "U2")
 					(unit 1)
@@
 			(effects (font (size 1.27 1.27)))
 		)
-		(property "Footprint" ""
+		(property "Footprint" "Resistor_SMD:R_0805_2012Metric"
 			(at 80.01 99.06 90)
 			(hide yes)
@@
 		(instances
 			(project "Flashover"
-				(path "/d341370c-bf24-48b8-b9fb-db9600491445/b4d4908f-d3cb-45c8-9e34-8e6e14bfce1f"
+				(path "/872055d3-e01a-4a82-8c05-28c93674a700/e0ce4150-4c2b-4816-bb42-05bac40058e5"
 					(reference "R16")
 					(unit 1)
@@
 			(effects (font (size 1.27 1.27)) (justify left))
 		)
-		(property "Footprint" ""
+		(property "Footprint" "Resistor_SMD:R_0805_2012Metric"
 			(at 71.12 106.68 0)
 			(hide yes)
@@
 		(instances
 			(project "Flashover"
-				(path "/d341370c-bf24-48b8-b9fb-db9600491445/b4d4908f-d3cb-45c8-9e34-8e6e14bfce1f"
+				(path "/872055d3-e01a-4a82-8c05-28c93674a700/e0ce4150-4c2b-4816-bb42-05bac40058e5"
 					(reference "R17")
 					(unit 1)
@@
 		(instances
 			(project "Flashover"
-				(path "/d341370c-bf24-48b8-b9fb-db9600491445/b4d4908f-d3cb-45c8-9e34-8e6e14bfce1f"
+				(path "/872055d3-e01a-4a82-8c05-28c93674a700/e0ce4150-4c2b-4816-bb42-05bac40058e5"
 					(reference "#PWR18")
 					(unit 1)
@@
 			(effects (font (size 1.27 1.27)) (justify right))
 		)
-		(property "Footprint" ""
+		(property "Footprint" "Package_SO:TSSOP-14_4.4x5mm_P0.65mm"
 			(at 137.16 93.98 0)
 			(hide yes)
@@
 		(instances
 			(project "Flashover"
-				(path "/d341370c-bf24-48b8-b9fb-db9600491445/b4d4908f-d3cb-45c8-9e34-8e6e14bfce1f"
+				(path "/872055d3-e01a-4a82-8c05-28c93674a700/e0ce4150-4c2b-4816-bb42-05bac40058e5"
 					(reference "U9")
 					(unit 1)
@@
 		(instances
 			(project "Flashover"
-				(path "/d341370c-bf24-48b8-b9fb-db9600491445/b4d4908f-d3cb-45c8-9e34-8e6e14bfce1f"
+				(path "/872055d3-e01a-4a82-8c05-28c93674a700/e0ce4150-4c2b-4816-bb42-05bac40058e5"
 					(reference "#PWR19")
 					(unit 1)
@@
 			(effects (font (size 1.27 1.27)))
 		)
-		(property "Footprint" ""
+		(property "Footprint" "Capacitor_SMD:C_1210_3225Metric"
 			(at 146.05 93.98 90)
 			(hide yes)
@@
 		(instances
 			(project "Flashover"
-				(path "/d341370c-bf24-48b8-b9fb-db9600491445/b4d4908f-d3cb-45c8-9e34-8e6e14bfce1f"
+				(path "/872055d3-e01a-4a82-8c05-28c93674a700/e0ce4150-4c2b-4816-bb42-05bac40058e5"
 					(reference "C9")
 					(unit 1)
@@
 			(effects (font (size 1.27 1.27)) (justify left))
 		)
-		(property "Footprint" ""
+		(property "Footprint" "Resistor_SMD:R_0805_2012Metric"
 			(at 154.94 102.87 0)
 			(hide yes)
@@
 		(instances
 			(project "Flashover"
-				(path "/d341370c-bf24-48b8-b9fb-db9600491445/b4d4908f-d3cb-45c8-9e34-8e6e14bfce1f"
+				(path "/872055d3-e01a-4a82-8c05-28c93674a700/e0ce4150-4c2b-4816-bb42-05bac40058e5"
 					(reference "R11")
 					(unit 1)
@@
 		(instances
 			(project "Flashover"
-				(path "/d341370c-bf24-48b8-b9fb-db9600491445/b4d4908f-d3cb-45c8-9e34-8e6e14bfce1f"
+				(path "/872055d3-e01a-4a82-8c05-28c93674a700/e0ce4150-4c2b-4816-bb42-05bac40058e5"
 					(reference "#PWR20")
 					(unit 1)
