File: pedals/distortion/kicad/Flashover/Flashover.kicad_pcb (KiCad board)
At the start: 4 copper layers, 87.6 x 84 mm, 95 parts, among them J1 Input, J2 Output, J3 9V DC, J4 SWD, J5 MIDI In, J6 MIDI Out, J7 To control board, K1 G6K-2F-Y 5VDC, K2 G6K-2F-Y 5VDC, Q1 MMBT3904, Q2 MMBT3904, SW5 Footswitch, U1 LM741, U11 H11L1, U2 TL072, U3 L7805, U4 RP2040, U5 W25Q16JVSS, U6 AP2112K-3.3, U7 MCP45HV51-104, U8 MCP45HV51-103, U9 MCP45HV51-103, Y1 12MHz

Commit message: Hand-route RUN and LED_EN on the Flashover main board; note progress
Co-Authored-By: Claude Opus 5.5 <noreply@anthropic.com>
Routing:
- net LED_EN: track 0.00 -> 55.6 mm, vias 0 -> 2
- net Net-(U4-RUN): track 0.00 -> 22.2 mm, vias 0 -> 2
Changed lines of the file:
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@@
 	)
 	(segment
+		(start 153.6 126.8)
+		(end 153.6 128.1325)
+		(width 0.2)
+		(layer "F.Cu")
+		(net "Net-(U4-RUN)")
+	)
+	(segment
+		(start 136.475 119.875)
+		(end 136.5 119.9)
+		(width 0.2)
+		(layer "F.Cu")
+		(net "Net-(U4-RUN)")
+	)
+	(segment
+		(start 153.6 128.1325)
+		(end 153.5475 128.185)
+		(width 0.2)
+		(layer "F.Cu")
+		(net "Net-(U4-RUN)")
+	)
+	(segment
+		(start 136.5 119.9)
+		(end 138.2 119.9)
+		(width 0.2)
+		(layer "F.Cu")
+		(net "Net-(U4-RUN)")
+	)
+	(segment
+		(start 136.475 119.1125)
+		(end 136.475 119.875)
+		(width 0.2)
+		(layer "F.Cu")
+		(net "Net-(U4-RUN)")
+	)
+	(via
+		(at 153.6 126.8)
+		(size 0.45)
+		(drill 0.2)
+		(layers "F.Cu" "B.Cu")
+		(net "Net-(U4-RUN)")
+	)
+	(via
+		(at 138.2 119.9)
+		(size 0.45)
+		(drill 0.2)
+		(layers "F.Cu" "B.Cu")
+		(net "Net-(U4-RUN)")
+	)
+	(segment
+		(start 145.1 126.8)
+		(end 153.6 126.8)
+		(width 0.2)
+		(layer "B.Cu")
+		(net "Net-(U4-RUN)")
+	)
+	(segment
+		(start 138.2 119.9)
+		(end 145.1 126.8)
+		(width 0.2)
+		(layer "B.Cu")
+		(net "Net-(U4-RUN)")
+	)
+	(segment
 		(start 146.285 81.695)
 		(end 147.5467 80.4333)
@@
 	)
 	(segment
+		(start 182.2 131.3)
+		(end 183.76 131.3)
+		(width 0.2)
+		(layer "F.Cu")
+		(net "LED_EN")
+	)
+	(segment
+		(start 183.76 131.3)
+		(end 185.86 133.4)
+		(width 0.2)
+		(layer "F.Cu")
+		(net "LED_EN")
+	)
+	(segment
+		(start 137.275 119.1125)
+		(end 137.6125 119.1125)
+		(width 0.2)
+		(layer "F.Cu")
+		(net "LED_EN")
+	)
+	(segment
+		(start 137.6125 119.1125)
+		(end 137.8 119.3)
+		(width 0.2)
+		(layer "F.Cu")
+		(net "LED_EN")
+	)
+	(via
+		(at 182.2 131.3)
+		(size 0.45)
+		(drill 0.2)
+		(layers "F.Cu" "B.Cu")
+		(net "LED_EN")
+	)
+	(via
+		(at 137.8 119.3)
+		(size 0.45)
+		(drill 0.2)
+		(layers "F.Cu" "B.Cu")
+		(net "LED_EN")
+	)
+	(segment
+		(start 137.8 118.806348)
+		(end 138.273748 118.3326)
+		(width 0.2)
+		(layer "B.Cu")
+		(net "LED_EN")
+	)
+	(segment
+		(start 138.273748 118.3326)
+		(end 139.140974 118.3326)
+		(width 0.2)
+		(layer "B.Cu")
+		(net "LED_EN")
+	)
+	(segment
+		(start 171.1029 120.2029)
+		(end 182.2 131.3)
+		(width 0.2)
+		(layer "B.Cu")
+		(net "LED_EN")
+	)
+	(segment
+		(start 139.140974 118.3326)
+		(end 141.011274 120.2029)
+		(width 0.2)
+		(layer "B.Cu")
+		(net "LED_EN")
+	)
+	(segment
+		(start 137.8 119.3)
+		(end 137.8 118.806348)
+		(width 0.2)
+		(layer "B.Cu")
+		(net "LED_EN")
+	)
+	(segment
+		(start 141.011274 120.2029)
+		(end 171.1029 120.2029)
+		(width 0.2)
+		(layer "B.Cu")
+		(net "LED_EN")
+	)
+	(segment
